File: KiCad Projects/GPIO_PROTECTION_RR/GPIO_PROTECTION_RR.kicad_sch (KiCad schematic)
At the start: 18 parts

Commit message: Working on design
Parts:
- removed D3: PESD3V3L2BT_215, PESD3V3L2BT:SOT95P230X110-3N, symbol PESD3V3L2BT_215:PESD3V3L2BT_215
- added C2: 470uF 25V, symbol Device:C_Polarized
- added C3: 10uF, symbol Device:C
- added C4: 0.1uF, symbol Device:C
- added D3: SMBJ14A, symbol Device:D_Zener
- added F1: 2A, symbol Device:Polyfuse
- added Q1: PMOS, symbol Simulation_SPICE:PMOS
- added R5, R9: 100k, symbol Device:R
- added U1: LM2596S-12, Package_TO_SOT_SMD:TO-263-5_TabPin3, symbol Regulator_Switching:LM2596S-12
Connections:
- net GND: now also C2.2, C3.2, C4.2, D3.2 (A), R9.2
- new net: Q1.1 (D), R5.1, R9.1
- new net: C2.1, C3.1, C4.1, D3.1 (K), R5.2
- new net: F1.2, Q1.3 (S)
- new net BAT+: F1.1
