File: KiCad Projects/FINAL_DESIGN/FINAL_DESIGN.kicad_sch (KiCad schematic)
At the start: 121 parts, among them U1 ESP32_NODEMCU

Commit message: Working on design
Parts:
- removed C21, C22, C23, C24, C27, C28, C29, C30: 100nf, Capacitor_SMD:C_0805_2012Metric, symbol Device:C
- removed D21, D22, D23, D24, D27, D28, D29, D30: D_Zener, Diode_SMD:D_SOD-882, symbol Device:D_Zener
- removed JP21, JP22, JP23, JP24, JP27, JP28, JP29, JP30: SolderJumper_2_Open, Jumper:SolderJumper-2_P1.3mm_Open_Pad1.0x1.5mm, symbol Jumper:SolderJumper_2_Open
- removed R21, R22, R23, R24, R27, R28, R29, R30: 150, RC0805FR-07330RL:RESC2012X60N, symbol RC0805FR-07330RL:RC0805FR-07330RL
- added C31, C32, C33, C34, C35, C36, C37, C38: 100nf, Capacitor_SMD:C_0805_2012Metric, symbol Device:C
- added D31, D32, D33, D34, D35, D36, D37, D38: D_Zener, Diode_SMD:D_SOD-882, symbol Device:D_Zener
- added J1, J2: Conn_01x19_Socket, Connector_PinHeader_2.54mm:PinHeader_1x19_P2.54mm_Vertical, symbol Connector:Conn_01x19_Socket
- added JP31, JP32, JP33, JP34, JP35, JP36, JP37, JP38: SolderJumper_2_Open, Jumper:SolderJumper-2_P1.3mm_Open_Pad1.0x1.5mm, symbol Jumper:SolderJumper_2_Open
- added R31, R32, R33, R34, R35, R36, R37, R38: 150, RC0805FR-07330RL:RESC2012X60N, symbol RC0805FR-07330RL:RC0805FR-07330RL
Connections:
- net ESP32_GPIO_0: no longer JP1.2 (B), R1.2
- net ESP32_GPIO_12: no longer JP10.2 (B), R10.2
- net ESP32_GPIO_13: no longer JP2.2 (B), R2.2
- net ESP32_GPIO_15: no longer JP4.2 (B), R4.2
- net ESP32_GPIO_17: no longer JP6.2 (B), R6.2
- net ESP32_GPIO_18: no longer JP18.2 (B), R18.2
- net ESP32_GPIO_19: no longer JP19.2 (B), R19.2
- net ESP32_GPIO_2: no longer JP7.2 (B), R7.2
- net ESP32_GPIO_21: no longer JP20.2 (B), R20.2
- net ESP32_GPIO_23: no longer JP13.2 (B), R13.2
- net ESP32_GPIO_25: no longer JP14.2 (B), R14.2
- net ESP32_GPIO_26: no longer JP15.2 (B), R15.2
- net ESP32_GPIO_27: no longer JP16.2 (B), R16.2
- net ESP32_GPIO_32: no longer JP11.2 (B), R11.2
- net ESP32_GPIO_33: no longer JP17.2 (B), R17.2
- net ESP32_GPIO_4: no longer JP8.2 (B), R8.2
- net ESP32_GPIO_5: no longer JP9.2 (B), R9.2
- net GND: now also C31.2, C32.2, C33.2, C34.2, C35.2, C36.2, C37.2, C38.2, D31.2 (A), D32.2 (A), D33.2 (A), D34.2 (A), D35.2 (A), D36.2 (A), D37.2 (A), D38.2 (A), J1.13 (Pin_13), J1.19 (Pin_19), J2.14 (Pin_14)
- net ESP32_GPIO renamed IO_34
- net IO_34: now also J2.5 (Pin_5); no longer JP26.2 (B), R26.2
- net ESP32_GPIO16 renamed IO16
- net ESP32_GPIO_14 renamed IO_14
- net IO_14: now also J2.12 (Pin_12)
- net ESP32_GPIO­_22 renamed IO­_22
- removed net EXT IN/OUT: D1.1 (K), D10.1 (K), D11.1 (K), D12.1 (K), D13.1 (K), D14.1 (K), D15.1 (K), D16.1 (K), D17.1 (K), D18.1 (K), D19.1 (K), D2.1 (K), D20.1 (K), D25.1 (K), D26.1 (K), D3.1 (K), D4.1 (K), D5.1 (K), D6.1 (K), D7.1 (K), D8.1 (K), D9.1 (K), R1.1, R10.1, R11.1, R12.1, R13.1, R14.1, R15.1, R16.1, R17.1, R18.1, R19.1, R2.1, R20.1, R25.1, R26.1, R3.1, R4.1, R5.1, R6.1, R7.1, R8.1, R9.1
- new net: C36.1, JP36.1 (A)
- new net: C35.1, JP35.1 (A)
- new net: C32.1, JP32.1 (A)
- new net: C34.1, JP34.1 (A)
- new net: C37.1, JP37.1 (A)
- new net: C38.1, JP38.1 (A)
- new net: C33.1, JP33.1 (A)
- new net: C31.1, JP31.1 (A)
- new net EN: J2.2 (Pin_2)
- new net GPIO_EXTERN_0: D1.1 (K), R1.1
- new net GPIO_EXTERN_1: D7.1 (K), R7.1
- new net GPIO_EXTERN_10: D37.1 (K), R37.1
- new net GPIO_EXTERN_11: D38.1 (K), R38.1
- new net GPIO_EXTERN_12: D10.1 (K), R10.1
- new net GPIO_EXTERN_13: D2.1 (K), R2.1
- new net GPIO_EXTERN_14: D3.1 (K), R3.1
- new net GPIO_EXTERN_15: D4.1 (K), R4.1
- new net GPIO_EXTERN_16: D5.1 (K), R5.1
- new net GPIO_EXTERN_17: D6.1 (K), R6.1
- new net GPIO_EXTERN_18: D18.1 (K), R18.1
- new net GPIO_EXTERN_19: D19.1 (K), R19.1
- new net GPIO_EXTERN_2: D8.1 (K), R8.1
- new net GPIO_EXTERN_21: D20.1 (K), R20.1
- new net GPIO_EXTERN_22: D12.1 (K), R12.1
- new net GPIO_EXTERN_23: D13.1 (K), R13.1
- new net GPIO_EXTERN_25: D14.1 (K), R14.1
- new net GPIO_EXTERN_26: D15.1 (K), R15.1
- new net GPIO_EXTERN_27: D16.1 (K), R16.1
- new net GPIO_EXTERN_3: D9.1 (K), R9.1
- new net GPIO_EXTERN_32: D11.1 (K), R11.1
- new net GPIO_EXTERN_33: D17.1 (K), R17.1
- new net GPIO_EXTERN_34: D25.1 (K), R25.1
- new net GPIO_EXTERN_35: D26.1 (K), R26.1
- new net GPIO_EXTERN_4: D31.1 (K), R31.1
- new net GPIO_EXTERN_5: D32.1 (K), R32.1
- new net GPIO_EXTERN_6: D33.1 (K), R33.1
- new net GPIO_EXTERN_7: D34.1 (K), R34.1
- new net GPIO_EXTERN_8: D35.1 (K), R35.1
- new net GPIO_EXTERN_9: D36.1 (K), R36.1
- new net IO_0: J1.6 (Pin_6), JP1.2 (B), R1.2
- new net IO_1: J1.16 (Pin_16), JP7.2 (B), R7.2
- new net IO_10: J2.17 (Pin_17), JP37.2 (B), R37.2
- new net IO_11: J2.18 (Pin_18), JP38.2 (B), R38.2
- new net IO_12: J2.13 (Pin_13), JP10.2 (B), R10.2
- new net IO_13: J2.15 (Pin_15), JP2.2 (B), R2.2
- new net IO_15: J1.4 (Pin_4), JP4.2 (B), R4.2
- new net IO_16: J1.8 (Pin_8)
- new net IO_17: J1.9 (Pin_9), JP6.2 (B), R6.2
- new net IO_18: J1.11 (Pin_11), JP18.2 (B), R18.2
- new net IO_19: J1.12 (Pin_12), JP19.2 (B), R19.2
- new net IO_2: J1.5 (Pin_5), JP8.2 (B), R8.2
- new net IO_21: J1.14 (Pin_14), JP20.2 (B), R20.2
- new net IO_22: J1.17 (Pin_17)
- new net IO_23: J1.18 (Pin_18), JP13.2 (B), R13.2
- new net IO_25: J2.9 (Pin_9), JP14.2 (B), R14.2
- new net IO_26: J2.10 (Pin_10), JP15.2 (B), R15.2
- new net IO_27: J2.11 (Pin_11), JP16.2 (B), R16.2
- new net IO_3: J1.15 (Pin_15), JP9.2 (B), R9.2
- new net IO_32: J2.7 (Pin_7), JP11.2 (B), R11.2
- new net IO_33: J2.8 (Pin_8), JP17.2 (B), R17.2
- new net IO_35: J2.6 (Pin_6), JP26.2 (B), R26.2
- new net IO_36: J2.3 (Pin_3)
- new net IO_39: J2.4 (Pin_4)
- new net IO_4: J1.7 (Pin_7), JP31.2 (B), R31.2
- new net IO_5: J1.10 (Pin_10), JP32.2 (B), R32.2
- new net IO_6: J1.1 (Pin_1), JP33.2 (B), R33.2
- new net IO_7: J1.2 (Pin_2), JP34.2 (B), R34.2
- new net IO_8: J1.3 (Pin_3), JP35.2 (B), R35.2
- new net IO_9: J2.16 (Pin_16), JP36.2 (B), R36.2
- new net VIN 5V: J2.19 (Pin_19)
Other:
- moved on the sheet: C10, C11, C12, C13, C14, C15, C16, C17, C18, C19, C2, C20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
