File: KiCad Projects/FINAL_DESIGN/FINAL_DESIGN.kicad_sch (KiCad schematic)
At the start: 146 parts, among them J1 Screw_Terminal_01x02, J2 Conn_01x19_Socket, J3 Conn_01x19_Socket, J4 Conn_01x19_Socket, J5 Conn_01x19_Socket, Q1 PMOS, U2 ESP32_NODEMCU

Commit message: changes
Parts:
- renumbered U2 to U1
Connections:
- net BUCK_OUT is gone; now on net CTRL_STG: C2.1, C4.1, C6.1, D2.2 (A)
- net BUCK_IN renamed CTRL_STG
Other:
- moved on the sheet: C1, C3, C5, D1

Commit message: Pcb design and stm code_x_lib worked
Parts:
- added C1: 680uF, Capacitor_THT:CP_Radial_D6.3mm_P2.50mm, symbol Device:C_Polarized
- added C2: 220uF, Capacitor_THT:CP_Radial_D6.3mm_P2.50mm, symbol Device:C_Polarized
- added D1: 1N5824, Diode_SMD:D_01005_0402Metric_Pad0.57x0.30mm_HandSolder, symbol Device:D
- added L1: WE-PD2_4532, Inductor_SMD:L_Wuerth_WE-PD2-Typ-MS, symbol WE-PD2_4532:WE-PD2_4532
- added U1: LM2596S-5, Package_TO_SOT_SMD:TO-263-5_TabPin3, symbol Regulator_Switching:LM2596S-5
- D2: renamed from D1; footprint Diode_THT:Diode_Bridge_Comchip_SCVB-L -> Diode_THT:D_5W_P10.16mm_Horizontal
- D3: renamed from D2; footprint Diode_THT:Diode_Bridge_Comchip_SCVB-L -> Diode_THT:D_DO-201_P15.24mm_Horizontal
- F1: value 2A -> 3A
- J1: footprint TerminalBlock_Dinkle:TerminalBlock_Dinkle_DT-55-B01X-02_P10.00mm -> TerminalBlock_4Ucon:TerminalBlock_4Ucon_1x02_P3.50mm_Vertical
- J4: footprint Connector_PinHeader_2.54mm:PinHeader_1x19_P2.54mm_Vertical -> Connector_PinSocket_2.54mm:PinSocket_1x19_P2.54mm_Vertical
- Q1: footprint Package_TO_SOT_SMD:SOT-23-6_Handsoldering -> Package_TO_SOT_THT:TO-92L_HandSolder
- renumbered C8 to C10, C9 to C11, C10 to C12, C11 to C13, C12 to C14, C13 to C15, C14 to C16, C15 to C17, C16 to C18, C17 to C19, C18 to C20, C19 to C21, C20 to C22, C21 to C23, C22 to C24, C23 to C25, C24 to C26, C25 to C27, C26 to C28, C27 to C29, C1 to C3, C28 to C30, C29 to C31, C30 to C32, C31 to C33, C32 to C34, C33 to C35, C34 to C36, C35 to C37, C36 to C38, C37 to C39, C3 to C4, C38 to C40, C2 to C5, C5 to C6, C4 to C7, C6 to C8, C7 to C9, D9 to D10, D10 to D11, D11 to D12, D12 to D13, D13 to D14, D14 to D15, D15 to D16, D16 to D17, D17 to D18, D18 to D19, D19 to D20, D20 to D21, D21 to D22, D22 to D23, D23 to D24, D24 to D25, D25 to D26, D26 to D27, D27 to D28, D28 to D29, D29 to D30, D30 to D31, D31 to D32, D32 to D33, D33 to D34, D34 to D35, D3 to D4, D4 to D5, D5 to D6, D6 to D7, D7 to D8, D8 to D9, U1 to U2
Connections:
- net GND: now also C1.2, C2.2, D1.2 (A), U1.3 (GND), U1.5 (~{ON}/OFF)
- net CTRL_STG renamed 12V
- net 12V: now also C1.1, U1.1 (VIN); no longer C5.1, C7.1, C8.1, D3.2 (A)
- new net: D1.1 (K), L1.1, U1.2 (OUT)
- new net 5V: C2.1, C5.1, C7.1, C8.1, D3.2 (A), L1.2, U1.4 (FB)
Other:
- moved on the sheet: C3, C4, C5, C6, C7, C8, D2, D3, F1, J1, Q1, R1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

Commit message: pcb
Parts:
- R2: value 100K -> 10K
Other:
- note added: "Note: All Capcitors 16V"
- note removed: "Note: All Capcitors 10V"
Changed lines of the file:
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@@
 		)
 	)
-	(text "Note:\nAll Capcitors 10V"
+	(text "Note:\nAll Capcitors 16V"
 		(exclude_from_sim no)
 		(at 111.252 61.468 0)
@@
 			)
 		)
-		(property "Value" "100K"
+		(property "Value" "10K"
 			(at 62.738 56.134 0)
 			(effects
