File: KiCad Projects/FINAL_DESIGN/FINAL_DESIGN.kicad_sch (KiCad schematic)
At the start: 147 parts, among them J1 Screw_Terminal_01x02, J2 Conn_01x19_Socket, J3 Conn_01x19_Socket, J4 Conn_01x19_Socket, J5 Conn_01x19_Socket, Q1 PMOS, U1 LM2596S-5, U2 ESP32_NODEMCU

Commit message: stm & pcb
Parts:
- added TP1: 12V, TestPoint:TestPoint_Pad_D1.5mm, symbol Connector:TestPoint
- added TP2: 3V3, TestPoint:TestPoint_Pad_D1.5mm, symbol Connector:TestPoint
- added TP3: 5V, TestPoint:TestPoint_Pad_D1.5mm, symbol Connector:TestPoint
- renumbered C16 to C15, C17 to C16, C18 to C17, C19 to C18, C20 to C19, C21 to C20, C22 to C21, C23 to C22, C24 to C23, C25 to C24, C26 to C25, C27 to C26, C28 to C27, C29 to C28, C30 to C29, C31 to C30, C32 to C31, C33 to C32, C34 to C33, C35 to C34, C36 to C35, C37 to C36, C38 to C37, C39 to C38, C40 to C39, D11 to D10, D12 to D11, D13 to D12, D14 to D13, D15 to D14, D16 to D15, D17 to D16, D18 to D17, D19 to D18, D20 to D19, D21 to D20, D22 to D21, D23 to D22, D24 to D23, D25 to D24, D26 to D25, D27 to D26, D28 to D27, D29 to D28, D30 to D29, D31 to D30, D32 to D31, D33 to D32, D34 to D33, D35 to D34, JP11 to JP10, JP12 to JP11, JP13 to JP12, JP14 to JP13, JP15 to JP14, JP16 to JP15, JP17 to JP16, JP18 to JP17, JP19 to JP18, JP20 to JP19, JP21 to JP20, JP22 to JP21, JP23 to JP22, JP24 to JP23, JP25 to JP24, JP26 to JP25, JP27 to JP26, JP28 to JP27, JP29 to JP28, JP30 to JP29, JP31 to JP30, JP32 to JP31, JP8 to JP7, JP9 to JP8, JP10 to JP9, R11 to R10, R12 to R11, R13 to R12, R14 to R13, R15 to R14, R16 to R15, R17 to R16, R18 to R17, R19 to R18, R20 to R19, R21 to R20, R22 to R21, R23 to R22, R24 to R23, R25 to R24, R26 to R25, R27 to R26, R28 to R27, R29 to R28, R30 to R29, R31 to R30, R32 to R31, R33 to R32, R34 to R33, R10 to R9
Connections:
- net +3V3: now also TP2.1
- net 12V: now also TP1.1
- net VIN 5V: now also TP3.1
