File: KiCad Projects/FINAL_DESIGN/FINAL_DESIGN.kicad_pcb (KiCad board)
At the start: 2 copper layers, 73.5 x 94.8 mm, 133 parts, among them J1 Conn_01x19_Socket, J2 Conn_01x19_Socket, J3 Conn_01x19_Socket, J4 Conn_01x19_Socket, U1 ESP32_NODEMCU

Commit message: Changes
Parts:
- added C1: 470uF, Capacitor_THT:CP_Radial_D6.3mm_P2.50mm, F.Cu at (-31.9, 45.1)
- added C2: 220uF, Capacitor_THT:CP_Radial_D6.3mm_P2.50mm, F.Cu at (-31.9, 53.0)
- added C3: 10uF, Capacitor_THT:C_Disc_D3.0mm_W2.0mm_P2.50mm, F.Cu at (-25.2, 43.0)
- added C4: 10uF, Capacitor_THT:C_Disc_D3.0mm_W2.0mm_P2.50mm, F.Cu at (-25.2, 46.5)
- added C5: 0.1uF, Capacitor_THT:C_Disc_D3.0mm_W1.6mm_P2.50mm, F.Cu at (-19.5, 42.8)
- added C6: 0.1uF, Capacitor_THT:C_Disc_D3.0mm_W1.6mm_P2.50mm, F.Cu at (-19.5, 46.0)
- added D1: D_Zener, Diode_THT:Diode_Bridge_Comchip_SCVB-L, F.Cu at (-60.5, 38.4)
- added D2: Shottky, Diode_THT:Diode_Bridge_Comchip_SCVB-L, F.Cu at (-60.5, 75.9)
- added F1: 2A, Fuse:FuseHolder_Blade_ATO_Littelfuse_FLR_178.6165, F.Cu at (-30.1, 36.0)
- added J1: Screw_Terminal_01x02, TerminalBlock_Dinkle:TerminalBlock_Dinkle_DT-55-B01X-02_P10.00mm, F.Cu at (78.0, 32.5)
- added Q1: PMOS, Package_TO_SOT_SMD:SOT-23-6_Handsoldering, F.Cu at (-19.1, 50.8)
- added R1: 100K, Resistor_SMD:R_0805_2012Metric_Pad1.20x1.40mm_HandSolder, F.Cu at (-24.4, 49.8)
- added R2: 100K, Resistor_SMD:R_0805_2012Metric_Pad1.20x1.40mm_HandSolder, F.Cu at (-24.4, 52.8)
- added U1: DC_DC_small, DC_DC_LM2596_small:DC_DC_LM2596_small, F.Cu at (114.5, 28.0)
- moved D25 134.4 mm to (81.5, 103.5), turned to -90 degrees
- moved C29 132.4 mm to (87.0, 107.5), turned to 180 degrees
- moved C27 131.7 mm to (73.0, 101.5)
- moved JP21 129.8 mm to (74.5, 97.3), turned to 90 degrees
- moved R25 129.3 mm to (87.0, 105.5)
- moved D24 127.9 mm to (81.3, 100.5), turned to 90 degrees
- moved JP23 127.6 mm to (90.5, 106.0), turned to 90 degrees
- moved JP26 126.4 mm to (123.0, 87.0), turned to 180 degrees
- moved C28 125.7 mm to (87.0, 103.5), turned to 180 degrees
- moved C32 124.9 mm to (126.5, 86.5)
- moved R24 122.8 mm to (87.0, 101.5)
- moved R23 122.7 mm to (81.5, 94.5), turned to 90 degrees
- moved D23 122.6 mm to (81.5, 91.5), turned to 90 degrees
- moved JP22 121.1 mm to (90.5, 102.5), turned to 90 degrees
- moved JP25 120.1 mm to (123.0, 84.5), turned to 180 degrees
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- renumbered C4 to C10, C5 to C11, C6 to C12, C7 to C13, C8 to C14, C9 to C15, C10 to C16, C11 to C17, C12 to C18, C13 to C19, C14 to C20, C15 to C21, C16 to C22, C17 to C23, C18 to C24, C19 to C25, C20 to C26, C21 to C27, C22 to C28, C23 to C29, C24 to C30, C25 to C31, C26 to C32, C27 to C33, C28 to C34, C29 to C35, C30 to C36, C31 to C37, C32 to C38, C1 to C7, C2 to C8, C3 to C9, D8 to D10, D9 to D11, D10 to D12, D11 to D13, D12 to D14, D13 to D15, D14 to D16, D15 to D17, D16 to D18, D17 to D19, D18 to D20, D19 to D21, D20 to D22, D21 to D23, D22 to D24, D23 to D25, D24 to D26, D25 to D27, D26 to D28, D27 to D29, D1 to D3, D28 to D30, D29 to D31, D30 to D32, D31 to D33, D32 to D34, D2 to D4, D3 to D5, D4 to D6, D5 to D7, D6 to D8, D7 to D9, J1 to J2, J2 to J4, J4 to J5, R8 to R10, R9 to R11, R10 to R12, R11 to R13, R12 to R14, R13 to R15, R14 to R16, R15 to R17, R16 to R18, R17 to R19, R18 to R20, R19 to R21, R20 to R22, R21 to R23, R22 to R24, R23 to R25, R24 to R26, R25 to R27, R26 to R28, R27 to R29, R1 to R3, R28 to R30, R29 to R31, R30 to R32, R31 to R33, R32 to R34, R2 to R4, R3 to R5, R4 to R6, R5 to R7, R6 to R8, R7 to R9, U1 to U2
Connections:
- JP22 pad 2: /IO­_22 -> /IO_22
- R24 pad 2: /IO­_22 -> /IO_22
Routing:
- net /RXD: track 5.88 -> 0.00 mm
- net /TXD: track 5.75 -> 0.00 mm
- net /IO_9: track 6.52 -> 2.69 mm

Commit message: changes
Parts:
- moved C5 6.37 mm to (-13.8, 45.5)
- moved C2 0.77 mm to (-32.5, 53.5)
- renumbered U2 to U1
Connections:
- C1 pad 1: BUCK_IN -> /CTRL_STG
- C2 pad 1: BUCK_OUT -> /CTRL_STG
- C3 pad 1: BUCK_IN -> /CTRL_STG
- C4 pad 1: BUCK_OUT -> /CTRL_STG
- C5 pad 1: BUCK_IN -> /CTRL_STG
- C6 pad 1: BUCK_OUT -> /CTRL_STG
- D1 pad 1: BUCK_IN -> /CTRL_STG
- D2 pad 2: BUCK_OUT -> /CTRL_STG
- Q1 pad 1: BUCK_IN -> /CTRL_STG
Changed lines of the file:
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@@
 	(net 122 "/ESP32_GPIO_32")
 	(net 123 "/ESP32_GPIO_21")
-	(net 124 "unconnected-(U2-GND_7-PadJ4_7)")
-	(net 125 "unconnected-(U2-5V-PadJ5_1)")
+	(net 124 "unconnected-(U1-GND_7-PadJ4_7)")
+	(net 125 "unconnected-(U1-5V-PadJ5_1)")
 	(net 126 "/ESP32_GPIO­_14")
 	(net 127 "/ESP32_GPIO_23")
 	(net 128 "/ESP32_GPIO_17")
 	(net 129 "/ESP32_GPIO­_3")
-	(net 130 "unconnected-(U2-EN-PadJ5_18)")
+	(net 130 "unconnected-(U1-EN-PadJ5_18)")
 	(net 131 "/ESP32_GPIO_13")
 	(net 132 "/ESP32_GPIO_12")
@@
 	(net 138 "/SN")
 	(net 139 "+3V3")
-	(net 140 "unconnected-(U2-3V3-PadJ5_19)")
-	(net 141 "unconnected-(U2-SP-PadJ5_17)")
-	(net 142 "unconnected-(U2-GND_1-PadJ4_1)")
-	(net 143 "unconnected-(U2-SN-PadJ5_16)")
-	(net 144 "unconnected-(U2-GND_6-PadJ5_6)")
+	(net 140 "unconnected-(U1-3V3-PadJ5_19)")
+	(net 141 "unconnected-(U1-SP-PadJ5_17)")
+	(net 142 "unconnected-(U1-GND_1-PadJ4_1)")
+	(net 143 "unconnected-(U1-SN-PadJ5_16)")
+	(net 144 "unconnected-(U1-GND_6-PadJ5_6)")
+	(net 145 "/CTRL_STG")
 	(footprint "Capacitor_SMD:C_0805_2012Metric"
 		(layer "F.Cu")
@@
 			(layers "*.Cu" "*.Mask")
 			(remove_unused_layers no)
-			(net 103 "BUCK_IN")
+			(net 145 "/CTRL_STG")
 			(pintype "passive")
 		)
@@
 			(remove_unused_layers no)
 			(roundrect_rratio 0.15625)
-			(net 103 "BUCK_IN")
+			(net 145 "/CTRL_STG")
 			(pintype "passive")
 		)
@@
 		(layer "F.Cu")
 		(at 232.5 60.5)
-		(property "Reference" "U2"
+		(property "Reference" "U1"
 			(at -11.075 -29.385 0)
 			(layer "F.SilkS")
@@
 			(layers "*.Cu" "*.Mask")
 			(remove_unused_layers no)
-			(net 142 "unconnected-(U2-GND_1-PadJ4_1)")
+			(net 142 "unconnected-(U1-GND_1-PadJ4_1)")
 			(pinfunction "GND_1")
 			(pintype "power_in")
@@
 			(layers "*.Cu" "*.Mask")
 			(remove_unused_layers no)
-			(net 124 "unconnected-(U2-GND_7-PadJ4_7)")
+			(net 124 "unconnected-(U1-GND_7-PadJ4_7)")
 			(pinfunction "GND_7")
 			(pintype "power_in")
@@
 			(layers "*.Cu" "*.Mask")
 			(remove_unused_layers no)
-			(net 125 "unconnected-(U2-5V-PadJ5_1)")
+			(net 125 "unconnected-(U1-5V-PadJ5_1)")
 			(pinfunction "5V")
 			(pintype "power_in")
@@
 			(layers "*.Cu" "*.Mask")
 			(remove_unused_layers no)
-			(net 144 "unconnected-(U2-GND_6-PadJ5_6)")
+			(net 144 "unconnected-(U1-GND_6-PadJ5_6)")
 			(pinfunction "GND_6")
 			(pintype "power_in")
@@
 			(layers "*.Cu" "*.Mask")
 			(remove_unused_layers no)
-			(net 143 "unconnected-(U2-SN-PadJ5_16)")
+			(net 143 "unconnected-(U1-SN-PadJ5_16)")
 			(pinfunction "SN")
 			(pintype "input")
@@
 			(layers "*.Cu" "*.Mask")
 			(remove_unused_layers no)
-			(net 141 "unconnected-(U2-SP-PadJ5_17)")
+			(net 141 "unconnected-(U1-SP-PadJ5_17)")
 			(pinfunction "SP")
 			(pintype "input")
@@
 			(layers "*.Cu" "*.Mask")
 			(remove_unused_layers no)
-			(net 130 "unconnected-(U2-EN-PadJ5_18)")
+			(net 130 "unconnected-(U1-EN-PadJ5_18)")
 			(pinfunction "EN")
 			(pintype "input")
@@
 			(layers "*.Cu" "*.Mask")
 			(remove_unused_layers no)
-			(net 140 "unconnected-(U2-3V3-PadJ5_19)")
+			(net 140 "unconnected-(U1-3V3-PadJ5_19)")
 			(pinfunction "3V3")
 			(pintype "power_in")
@@
 			(layers "*.Cu" "*.Mask")
 			(remove_unused_layers no)
-			(net 103 "BUCK_IN")
+			(net 145 "/CTRL_STG")
 			(pinfunction "K")
 			(pintype "passive")
@@
 			(layers "F.Cu" "F.Mask" "F.Paste")
 			(roundrect_rratio 0.25)
-			(net 103 "BUCK_IN")
+			(net 145 "/CTRL_STG")
 			(pinfunction "D")
 			(pintype "passive")
@@
 			(layers "*.Cu" "*.Mask")
 			(remove_unused_layers no)
-			(net 104 "BUCK_OUT")
+			(net 145 "/CTRL_STG")
 			(pintype "passive")
 		)
@@
 			(remove_unused_layers no)
 			(roundrect_rratio 0.25)
-			(net 104 "BUCK_OUT")
+			(net 145 "/CTRL_STG")
 			(pinfunction "A")
 			(pintype "passive")
@@
 	(footprint "Capacitor_THT:CP_Radial_D6.3mm_P2.50mm"
 		(layer "F.Cu")
-		(at -31.914759 53)
+		(at -32.5 53.5)
 		(descr "CP, Radial series, Radial, pin pitch=2.50mm, diameter=6.3mm, height=7mm, Electrolytic Capacitor")
 		(tags "CP Radial series Radial pin pitch 2.50mm diameter 6.3mm height 7mm Electrolytic Capacitor")
@@
 			(remove_unused_layers no)
 			(roundrect_rratio 0.15625)
-			(net 104 "BUCK_OUT")
+			(net 145 "/CTRL_STG")
 			(pintype "passive")
 		)
@@
 			(layers "*.Cu" "*.Mask")
 			(remove_unused_layers no)
-			(net 104 "BUCK_OUT")
+			(net 145 "/CTRL_STG")
 			(pintype "passive")
 		)
@@
 	(footprint "Capacitor_THT:C_Disc_D3.0mm_W1.6mm_P2.50mm"
 		(layer "F.Cu")
-		(at -19.52 42.8)
+		(at -13.75 45.5)
 		(descr "C, Disc series, Radial, pin pitch=2.50mm, diameter*width=3.0*1.6mm^2, Capacitor, http://www.vishay.com/docs/45233/krseries.pdf")
 		(tags "C Disc series Radial pin pitch 2.50mm diameter 3.0mm width 1.6mm Capacitor")
@@
 			(layers "*.Cu" "*.Mask")
 			(remove_unused_layers no)
-			(net 103 "BUCK_IN")
+			(net 145 "/CTRL_STG")
 			(pintype "passive")
 		)

Commit message: Pcb design and stm code_x_lib worked
Parts:
- added C1: 680uF, Capacitor_THT:CP_Radial_D6.3mm_P2.50mm, F.Cu at (26.7, 99.2)
- added C2: 220uF, Capacitor_THT:CP_Radial_D6.3mm_P2.50mm, F.Cu at (24.4, 92.3)
- added D1: 1N5824, Diode_SMD:D_01005_0402Metric_Pad0.57x0.30mm_HandSolder, F.Cu at (35.4, 100.3)
- added D35: 1N5824, Diode_SMD:D_SOD-123F, F.Cu at (34.6, 96.2)
- added L1: WE-PD2_4532, Inductor_SMD:L_Wuerth_WE-PD2-Typ-MS, F.Cu at (35.6, 91.0)
- D2: renamed from D1; footprint Diode_THT:Diode_Bridge_Comchip_SCVB-L -> Diode_THT:D_5W_P10.16mm_Horizontal
- D3: renamed from D2; footprint Diode_THT:Diode_Bridge_Comchip_SCVB-L -> Diode_THT:D_DO-201_P15.24mm_Horizontal
- F1: value 2A -> 3A
- J1: footprint TerminalBlock_Dinkle:TerminalBlock_Dinkle_DT-55-B01X-02_P10.00mm -> TerminalBlock_4Ucon:TerminalBlock_4Ucon_1x02_P3.50mm_Vertical
- J2, J4: footprint Connector_PinHeader_2.54mm:PinHeader_1x19_P2.54mm_Vertical -> Connector_PinSocket_2.54mm:PinSocket_1x19_P2.54mm_Vertical
- Q1: footprint Package_TO_SOT_SMD:SOT-23-6_Handsoldering -> Package_TO_SOT_THT:TO-92L_HandSolder
- U1: value DC_DC_small -> LM2596S-5; footprint DC_DC_LM2596_small:DC_DC_LM2596_small -> Package_TO_SOT_SMD:TO-263-5_TabPin3
- moved D2 177.9 mm to (116.4, 19.9), turned to -90 degrees
- moved C3 156.3 mm to (122.5, 21.0)
- moved C4 148.8 mm to (122.8, 26.5)
- moved C5 144.9 mm to (112.0, 42.5)
- moved R2 137.2 mm to (110.0, 25.0), turned to 180 degrees
- moved Q1 135.0 mm to (112.3, 19.5), turned to 180 degrees
- moved F1 121.8 mm to (90.5, 19.0)
- moved U1 96.1 mm to (34.6, 81.3)
- moved C7 61.7 mm to (35.6, 36.1)
- moved C6 61.7 mm to (47.0, 35.0)
- moved C8 61.7 mm to (41.3, 35.5)
- moved R1 61.7 mm to (36.4, 39.4)
- moved D3 41.8 mm to (-18.9, 80.7)
- moved J1 10.5 mm to (77.5, 22.0), turned to -90 degrees
- moved J2 0.20 mm to (94.0, 60.6)
- renumbered C8 to C10, C9 to C11, C10 to C12, C11 to C13, C12 to C14, C13 to C15, C14 to C16, C15 to C17, C16 to C18, C17 to C19, C18 to C20, C19 to C21, C20 to C22, C21 to C23, C22 to C24, C23 to C25, C24 to C26, C25 to C27, C26 to C28, C27 to C29, C1 to C3, C28 to C30, C29 to C31, C30 to C32, C31 to C33, C32 to C34, C33 to C35, C34 to C36, C35 to C37, C36 to C38, C37 to C39, C3 to C4, C38 to C40, C2 to C5, C5 to C6, C4 to C7, C6 to C8, C7 to C9, D9 to D10, D10 to D11, D11 to D12, D12 to D13, D13 to D14, D14 to D15, D15 to D16, D16 to D17, D17 to D18, D18 to D19, D19 to D20, D20 to D21, D21 to D22, D22 to D23, D23 to D24, D24 to D25, D25 to D26, D26 to D27, D27 to D28, D28 to D29, D29 to D30, D30 to D31, D31 to D32, D32 to D33, D33 to D34, D34 to D35, D3 to D4, D4 to D5, D5 to D6, D6 to D7, D7 to D8, D8 to D9, U1 to U2
Connections:
- C3 pad 1: /CTRL_STG -> /12V
- C4 pad 1: /CTRL_STG -> /12V
- C5 pad 1: /CTRL_STG -> /5V
- C6 pad 1: /CTRL_STG -> /12V
- C7 pad 1: /CTRL_STG -> /5V
- C8 pad 1: /CTRL_STG -> /5V
- D2 pad 1: /CTRL_STG -> /12V
- D3 pad 2: /CTRL_STG -> /5V
- Q1 pad 1: /CTRL_STG -> /12V
- U1 pad 1: BUCK_IN -> /12V
- U1 pad 2: GND -> Net-(D1-K)
- U1 pad 3: BUCK_OUT -> GND
- U1 pad 4: GND -> /5V

Commit message: pcb
Parts:
- removed the D35 at (34.6, 96.2)
- R2: value 100K -> 10K
- moved D3 159.8 mm to (138.5, 53.2), turned to 90 degrees
- moved C2 106.5 mm to (104.0, 21.5), turned to 180 degrees
- moved D1 98.5 mm to (101.9, 27.5), turned to 180 degrees
- moved C1 93.8 mm to (96.0, 36.0), turned to 180 degrees
- moved L1 89.8 mm to (95.4, 24.0), turned to 180 degrees
- moved C7 79.1 mm to (114.0, 25.5), turned to 180 degrees
- moved R1 76.4 mm to (112.5, 32.0), turned to 180 degrees
- moved C8 75.2 mm to (115.0, 20.5), turned to 180 degrees
- moved U1 72.8 mm to (81.6, 25.7), turned to 180 degrees
- moved J1 57.9 mm to (135.4, 23.2), turned to 90 degrees
- moved F1 48.0 mm to (137.0, 31.0), turned to 180 degrees
- moved C6 37.5 mm to (84.2, 39.8), turned to -90 degrees
- moved C3 36.6 mm to (94.0, 44.0), turned to 180 degrees
- moved C4 35.1 mm to (90.0, 39.0), turned to 180 degrees
- moved D2 29.2 mm to (101.6, 45.1), turned to 90 degrees
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