File: KiCad Projects/FINAL_DESIGN/FINAL_DESIGN.kicad_pcb (KiCad board)
At the start: 2 copper layers, 73.5 x 94.8 mm, 152 parts, among them J1 Screw_Terminal_01x02, J2 Conn_01x19_Socket, J3 Conn_01x19_Socket, J4 Conn_01x19_Socket, J5 Conn_01x19_Socket, Q1 PMOS, U1 LM2596S-5, U2 ESP32_NODEMCU

Commit message: work
Parts:
- removed R8: 150, RC0805FR-07330RL:RESC2012X60N
- moved C6 27.1 mm to (74.0, 38.0)
- moved JP21 18.9 mm to (92.9, 93.0)
- moved D12 14.5 mm to (85.5, 72.8)
- moved D21 12.5 mm to (85.5, 68.9), turned to 0 degrees
- moved JP9 11.1 mm to (79.8, 66.3)
- moved C27 11.0 mm to (80.0, 79.8)
- moved R23 10.6 mm to (80.5, 84.0)
- moved R11 9.76 mm to (79.7, 63.3)
- moved C29 9.56 mm to (80.2, 95.1)
- moved C25 9.49 mm to (106.9, 81.8)
- moved C17 7.83 mm to (80.2, 69.6)
- moved J3 5.28 mm to (73.4, 58.8)
- moved R21 5.20 mm to (89.3, 84.9)
- moved R22 5.20 mm to (89.3, 86.9)
- moved JP17 4.97 mm to (92.9, 75.7)
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Routing:
- net /IO_4: track 6.08 -> 0.00 mm
- net /IO_0: track 5.78 -> 0.65 mm
- net /IO_3: track 6.09 -> 1.41 mm
- net /IO_1: track 5.78 -> 1.14 mm
- net /IO_2: track 6.34 -> 1.80 mm
- net GND: track 13.1 -> 10.2 mm, vias 12 -> 10
- net Net-(JP1-A): track 2.42 -> 0.08 mm
- net Net-(JP2-A): track 2.19 -> 0.00 mm
- net Net-(JP4-A): track 2.40 -> 1.20 mm
- net /I/O_4: track 1.07 -> 0.00 mm
Other:
- board size 73.5 x 94.8 mm -> 82 x 94.8 mm

Commit message: PCB
Parts:
- moved C25 17.5 mm to (89.5, 83.0), turned to 0 degrees
- moved C30 0.65 mm to (89.5, 101.7)
- moved C31 0.65 mm to (89.5, 105.7)
- moved R24 0.65 mm to (89.5, 99.7)
- moved R25 0.65 mm to (89.5, 103.7)
- moved C10 0.65 mm to (89.5, 95.6)
- moved C12 0.65 mm to (89.5, 91.6)
- moved C28 0.65 mm to (89.5, 89.5)
- moved R21 0.65 mm to (89.5, 85.5)
- moved R22 0.65 mm to (89.5, 87.5)
- moved R4 0.65 mm to (89.5, 97.6)
- moved R6 0.65 mm to (89.5, 93.6)
Changed lines of the file:
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@@
 		(tags "Diode SOD882 DFN1006-2")
 		(property "Reference" "D26"
-			(at -1.25 0 90)
+			(at -1.495 -0.6 90)
 			(layer "F.SilkS")
 			(effects
@@
 	(footprint "RC0805FR-07330RL:RESC2012X60N"
 		(layer "F.Cu")
-		(at 89.3 97)
+		(at 89.545 97.6)
 		(property "Reference" "R4"
 			(at -0.3 0.5 0)
@@
 		(tags "solder jumper open")
 		(property "Reference" "JP19"
-			(at 0 -1.8 90)
+			(at -0.6 -1.555 90)
 			(layer "F.SilkS")
 			(effects
@@
 	(footprint "RC0805FR-07330RL:RESC2012X60N"
 		(layer "F.Cu")
-		(at 89.3 99.1)
+		(at 89.545 99.7)
 		(property "Reference" "R24"
 			(at 0.29 -1.87 0)
@@
 	(footprint "Capacitor_SMD:C_0805_2012Metric"
 		(layer "F.Cu")
-		(at 89.3 88.9 180)
+		(at 89.545 89.5 180)
 		(descr "Capacitor SMD 0805 (2012 Metric), square (rectangular) end terminal, IPC-7351 nominal, (Body size source: IPC-SM-782 page 76, https://www.pcb-3d.com/wordpress/wp-content/uploads/ipc-sm-782a_amendment_1_and_2.pdf, https://docs.google.com/spreadsheets/d/1BsfQQcO9C6DZCsRaXUlFlo91Tg2WpOkGARC1WS5S8t0/edit?usp=sharing), generated with kicad-footprint-generator")
 		(tags "capacitor")
@@
 	(footprint "Capacitor_SMD:C_0805_2012Metric"
 		(layer "F.Cu")
-		(at 89.3 95 180)
+		(at 89.545 95.6 180)
 		(descr "Capacitor SMD 0805 (2012 Metric), square (rectangular) end terminal, IPC-7351 nominal, (Body size source: IPC-SM-782 page 76, https://www.pcb-3d.com/wordpress/wp-content/uploads/ipc-sm-782a_amendment_1_and_2.pdf, https://docs.google.com/spreadsheets/d/1BsfQQcO9C6DZCsRaXUlFlo91Tg2WpOkGARC1WS5S8t0/edit?usp=sharing), generated with kicad-footprint-generator")
 		(tags "capacitor")
@@
 	(footprint "RC0805FR-07330RL:RESC2012X60N"
 		(layer "F.Cu")
-		(at 89.3 93)
+		(at 89.545 93.6)
 		(property "Reference" "R6"
 			(at -2.5 0 0)
@@
 	(footprint "Capacitor_SMD:C_0805_2012Metric"
 		(layer "F.Cu")
-		(at 89.3 101.1 180)
+		(at 89.545 101.7 180)
 		(descr "Capacitor SMD 0805 (2012 Metric), square (rectangular) end terminal, IPC-7351 nominal, (Body size source: IPC-SM-782 page 76, https://www.pcb-3d.com/wordpress/wp-content/uploads/ipc-sm-782a_amendment_1_and_2.pdf, https://docs.google.com/spreadsheets/d/1BsfQQcO9C6DZCsRaXUlFlo91Tg2WpOkGARC1WS5S8t0/edit?usp=sharing), generated with kicad-footprint-generator")
 		(tags "capacitor")
@@
 	(footprint "RC0805FR-07330RL:RESC2012X60N"
 		(layer "F.Cu")
-		(at 89.3 103.1)
+		(at 89.545 103.7)
 		(property "Reference" "R25"
 			(at -0.41 -1.27 0)
@@
 	(footprint "Capacitor_SMD:C_0805_2012Metric"
 		(layer "F.Cu")
-		(at 89.3 91 180)
+		(at 89.545 91.6 180)
 		(descr "Capacitor SMD 0805 (2012 Metric), square (rectangular) end terminal, IPC-7351 nominal, (Body size source: IPC-SM-782 page 76, https://www.pcb-3d.com/wordpress/wp-content/uploads/ipc-sm-782a_amendment_1_and_2.pdf, https://docs.google.com/spreadsheets/d/1BsfQQcO9C6DZCsRaXUlFlo91Tg2WpOkGARC1WS5S8t0/edit?usp=sharing), generated with kicad-footprint-generator")
 		(tags "capacitor")
@@
 		(tags "solder jumper open")
 		(property "Reference" "JP21"
-			(at 0 -1.8 90)
+			(at -0.6 -1.555 90)
 			(layer "F.SilkS")
 			(effects
@@
 		(tags "solder jumper open")
 		(property "Reference" "JP20"
-			(at 0.48 -2 90)
+			(at -0.12 -1.755 90)
 			(layer "F.SilkS")
 			(effects
@@
 	(footprint "RC0805FR-07330RL:RESC2012X60N"
 		(layer "F.Cu")
-		(at 89.255 86.9)
+		(at 89.5 87.5)
 		(property "Reference" "R22"
 			(at 0.855 1.62 0)
@@
 	(footprint "Capacitor_SMD:C_0805_2012Metric"
 		(layer "F.Cu")
-		(at 89.3 105.1 180)
+		(at 89.545 105.7 180)
 		(descr "Capacitor SMD 0805 (2012 Metric), square (rectangular) end terminal, IPC-7351 nominal, (Body size source: IPC-SM-782 page 76, https://www.pcb-3d.com/wordpress/wp-content/uploads/ipc-sm-782a_amendment_1_and_2.pdf, https://docs.google.com/spreadsheets/d/1BsfQQcO9C6DZCsRaXUlFlo91Tg2WpOkGARC1WS5S8t0/edit?usp=sharing), generated with kicad-footprint-generator")
 		(tags "capacitor")
@@
 	(footprint "RC0805FR-07330RL:RESC2012X60N"
 		(layer "F.Cu")
-		(at 89.255 84.9)
+		(at 89.5 85.5)
 		(property "Reference" "R21"
 			(at -3.055 -0.95 0)
@@
 	(footprint "Capacitor_SMD:C_0805_2012Metric"
 		(layer "F.Cu")
-		(at 106.9 81.78 -90)
+		(at 89.45 83)
 		(descr "Capacitor SMD 0805 (2012 Metric), square (rectangular) end terminal, IPC-7351 nominal, (Body size source: IPC-SM-782 page 76, https://www.pcb-3d.com/wordpress/wp-content/uploads/ipc-sm-782a_amendment_1_and_2.pdf, https://docs.google.com/spreadsheets/d/1BsfQQcO9C6DZCsRaXUlFlo91Tg2WpOkGARC1WS5S8t0/edit?usp=sharing), generated with kicad-footprint-generator")
 		(tags "capacitor")
 		(property "Reference" "C25"
-			(at 0 -1.68 90)
+			(at 0 -1.68 0)
 			(layer "F.SilkS")
 			(effects
@@
 		)
 		(property "Value" "100nf"
-			(at 0 1.68 90)
+			(at 0 1.68 0)
 			(layer "F.Fab")
 			(effects
@@
 		)
 		(property "Datasheet" "~"
-			(at 0 0 90)
+			(at 0 0 0)
 			(layer "F.Fab")
 			(hide yes)
@@
 		)
 		(property "Description" "Unpolarized capacitor"
-			(at 0 0 90)
+			(at 0 0 0)
 			(layer "F.Fab")
 			(hide yes)
@@
 		)
 		(property "Assembly" "DNP"
-			(at 0 0 270)
+			(at 0 0 0)
 			(unlocked yes)
 			(layer "F.Fab")
@@
 		(attr smd dnp)
 		(fp_line
-			(start -0.261252 0.735)
-			(end 0.261252 0.735)
+			(start -0.261252 -0.735)
+			(end 0.261252 -0.735)
 			(stroke
 				(width 0.12)
@@
 		)
 		(fp_line
-			(start -0.261252 -0.735)
-			(end 0.261252 -0.735)
+			(start -0.261252 0.735)
+			(end 0.261252 0.735)
 			(stroke
 				(width 0.12)
@@
 		)
 		(fp_text user "${REFERENCE}"
-			(at 0 0 90)
+			(at 0 0 0)
 			(layer "F.Fab")
 			(effects
@@
 		)
 		(pad "1" smd roundrect
-			(at -0.95 0 270)
+			(at -0.95 0)
 			(size 1 1.45)
 			(layers "F.Cu" "F.Mask" "F.Paste")
@@
 		)
 		(pad "2" smd roundrect
-			(at 0.95 0 270)
+			(at 0.95 0)
 			(size 1 1.45)
 			(layers "F.Cu" "F.Mask" "F.Paste")
@@
 		(tags "Diode SOD882 DFN1006-2")
 		(property "Reference" "D24"
-			(at 1.25 0 90)
+			(at 1.495 0.6 90)
 			(layer "F.SilkS")
 			(effects
@@
 	)
 	(segment
-		(start 88.35 95)
-		(end 87.3 95)
+		(start 88.595 95.6)
+		(end 87.545 95.6)
 		(width 0.2)
 		(layer "F.Cu")
@@
 	)
 	(segment
-		(start 87.3 91)
-		(end 88.35 91)
+		(start 87.545 91.6)
+		(end 88.595 91.6)
 		(width 0.2)
 		(layer "F.Cu")
@@
 	)
 	(via
-		(at 87.2 91.4)
+		(at 87.445 92)
 		(size 0.6)
 		(drill 0.3)
@@
 	)
 	(via
-		(at 87.2 95.4)
+		(at 87.445 96)
 		(size 0.6)
 		(drill 0.3)
@@
 	)
 	(segment
-		(start 90.25 91)
-		(end 91.1 91.85)
+		(start 90.495 91.6)
+		(end 91.345 92.45)
 		(width 0.2)
 		(layer "F.Cu")

Commit message: work
Parts:
- moved R18 21.8 mm to (79.7, 65.8)
- moved R23 8.81 mm to (85.0, 91.5), turned to 180 degrees
- moved C27 8.50 mm to (85.3, 86.5), turned to 180 degrees
- moved R20 5.86 mm to (85.2, 78.8), turned to 0 degrees
- moved JP9 5.64 mm to (85.1, 64.2), turned to 180 degrees
- moved C29 5.55 mm to (85.7, 95.2), turned to 180 degrees
- moved JP16 5.04 mm to (105.2, 65.2)
- moved C17 3.22 mm to (82.8, 67.7), turned to -90 degrees
- moved J3 2.68 mm to (76.0, 58.1)
- moved D23 2.25 mm to (85.4, 84.8)
- moved D22 2.15 mm to (85.3, 82.8)
- moved D11 1.30 mm to (85.7, 61.8)
- moved D7 0.58 mm to (85.7, 93.5)
- moved JP1 0.20 mm to (92.9, 68.3)
- moved JP17 0.20 mm to (92.9, 75.5)
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Routing:
- net GND: track 10.2 -> 7.33 mm, vias 10 -> 5

Commit message: work
Parts:
- moved D19 19.7 mm to (82.7, 66.0)
- moved R18 5.71 mm to (82.0, 60.5), turned to 180 degrees
- moved C17 1.27 mm to (82.5, 69.0)
Routing:
- net GND: track 7.33 -> 5.46 mm, vias 5 -> 4
Changed lines of the file:
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@@
 	(footprint "Diode_SMD:D_SOD-882"
 		(layer "F.Cu")
-		(at 101.505 60.38)
+		(at 82.65 66)
 		(descr "SOD-882, DFN1006-2, body 1.0 x 0.6 x 0.48mm, pitch 0.65mm, https://assets.nexperia.com/documents/package-information/SOD882.pdf")
 		(tags "Diode SOD882 DFN1006-2")
@@
 	(footprint "RC0805FR-07330RL:RESC2012X60N"
 		(layer "F.Cu")
-		(at 79.705 65.75)
+		(at 81.955 60.5 180)
 		(property "Reference" "R18"
 			(at -0.41 -1.27 0)
@@
 		(attr smd)
 		(fp_line
-			(start -0.17 -0.68)
-			(end 0.17 -0.68)
+			(start -0.17 0.68)
+			(end 0.17 0.68)
 			(stroke
 				(width 0.127)
@@
 		)
 		(fp_line
-			(start -0.17 0.68)
-			(end 0.17 0.68)
+			(start -0.17 -0.68)
+			(end 0.17 -0.68)
 			(stroke
 				(width 0.127)
@@
 		)
 		(fp_line
-			(start -1.665 -0.94)
+			(start 1.665 0.94)
 			(end 1.665 -0.94)
 			(stroke
@@
 		(fp_line
 			(start -1.665 0.94)
-			(end -1.665 -0.94)
+			(end 1.665 0.94)
 			(stroke
 				(width 0.05)
@@
 		(fp_line
 			(start -1.665 0.94)
-			(end 1.665 0.94)
+			(end -1.665 -0.94)
 			(stroke
 				(width 0.05)
@@
 		)
 		(fp_line
-			(start 1.665 0.94)
+			(start -1.665 -0.94)
 			(end 1.665 -0.94)
 			(stroke
@@
 		)
 		(fp_line
-			(start -1.05 0.68)
-			(end -1.05 -0.68)
+			(start 1.05 0.68)
+			(end 1.05 -0.68)
 			(stroke
 				(width 0.127)
@@
 		)
 		(fp_line
-			(start 1.05 -0.68)
-			(end -1.05 -0.68)
+			(start 1.05 0.68)
+			(end -1.05 0.68)
 			(stroke
 				(width 0.127)
@@
 		)
 		(fp_line
-			(start 1.05 0.68)
-			(end -1.05 0.68)
+			(start 1.05 -0.68)
+			(end -1.05 -0.68)
 			(stroke
 				(width 0.127)
@@
 		)
 		(fp_line
-			(start 1.05 0.68)
-			(end 1.05 -0.68)
+			(start -1.05 0.68)
+			(end -1.05 -0.68)
 			(stroke
 				(width 0.127)
@@
 		)
 		(pad "1" smd rect
-			(at -0.955 0)
+			(at -0.955 0 180)
 			(size 0.92 1.38)
 			(layers "F.Cu" "F.Mask" "F.Paste")
@@
 		)
 		(pad "2" smd rect
-			(at 0.955 0)
+			(at 0.955 0 180)
 			(size 0.92 1.38)
 			(layers "F.Cu" "F.Mask" "F.Paste")
@@
 	(footprint "Capacitor_SMD:C_0805_2012Metric"
 		(layer "F.Cu")
-		(at 82.75 67.7 -90)
+		(at 82.5 68.95 -90)
 		(descr "Capacitor SMD 0805 (2012 Metric), square (rectangular) end terminal, IPC-7351 nominal, (Body size source: IPC-SM-782 page 76, https://www.pcb-3d.com/wordpress/wp-content/uploads/ipc-sm-782a_amendment_1_and_2.pdf, https://docs.google.com/spreadsheets/d/1BsfQQcO9C6DZCsRaXUlFlo91Tg2WpOkGARC1WS5S8t0/edit?usp=sharing), generated with kicad-footprint-generator")
 		(tags "capacitor")
@@
 	)
 	(segment
-		(start 82.255 74.2)
-		(end 82.205 74.25)
-		(width 0.2)
-		(layer "F.Cu")
-		(net 2)
-	)
-	(segment
-		(start 83.255 73.5)
-		(end 83.255 72.7)
-		(width 0.2)
-		(layer "F.Cu")
-		(net 2)
-	)
-	(segment
-		(start 83.255 74.2)
-		(end 82.255 74.2)
-		(width 0.2)
-		(layer "F.Cu")
-		(net 2)
-	)
-	(segment
 		(start 88.595 95.6)
 		(end 87.545 95.6)
@@
 		(size 0.6)
 		(drill 0.3)
-		(layers "F.Cu" "B.Cu")
-		(free yes)
-		(net 2)
-	)
-	(via
-		(at 83.255 72.7)
-		(size 0.6)
-		(drill 0.3)

Commit message: stm & pcb
Parts:
- removed D35: 1N5824, Diode_SMD:D_SOD-123F
- added R8: 150, RC0805FR-07330RL:RESC2012X60N, F.Cu at (82.6, 92.8)
- added TP1: 12V, TestPoint:TestPoint_Pad_D1.5mm, F.Cu at (104.8, 44.4)
- added TP2: 3V3, TestPoint:TestPoint_Pad_D1.5mm, F.Cu at (128.7, 66.4)
- added TP3: 5V, TestPoint:TestPoint_Pad_D1.5mm, F.Cu at (141.8, 47.4)
- moved D3 163.4 mm to (141.9, 51.8), turned to 180 degrees
- moved C2 90.1 mm to (105.5, 53.0), turned to 90 degrees
- moved C7 88.0 mm to (122.0, 53.0), turned to 90 degrees
- moved C8 79.7 mm to (119.0, 53.0), turned to 90 degrees
- moved C1 77.6 mm to (81.7, 44.5), turned to 180 degrees
- moved L1 74.5 mm to (103.6, 60.5), turned to 90 degrees
- moved R1 74.2 mm to (110.2, 31.1), turned to 90 degrees
- moved D1 74.2 mm to (98.6, 61.3), turned to 180 degrees
- moved U1 65.8 mm to (91.7, 48.6), turned to 90 degrees
- moved J1 62.9 mm to (138.1, 38.9), turned to 90 degrees
- moved F1 42.4 mm to (127.8, 39.1), turned to 180 degrees
- moved C4 39.0 mm to (84.8, 35.8), turned to -90 degrees
- moved C3 32.8 mm to (93.2, 35.6), turned to -90 degrees
- moved D2 22.6 mm to (100.3, 35.9)
- moved D20 21.6 mm to (79.6, 89.7), turned to -90 degrees
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- renumbered C16 to C15, C17 to C16, C18 to C17, C19 to C18, C20 to C19, C21 to C20, C22 to C21, C23 to C22, C24 to C23, C25 to C24, C26 to C25, C27 to C26, C28 to C27, C29 to C28, C30 to C29, C31 to C30, C32 to C31, C33 to C32, C34 to C33, C35 to C34, C36 to C35, C37 to C36, C38 to C37, C39 to C38, C40 to C39, D11 to D10, D12 to D11, D13 to D12, D14 to D13, D15 to D14, D16 to D15, D17 to D16, D18 to D17, D19 to D18, D20 to D19, D21 to D20, D22 to D21, D23 to D22, D24 to D23, D25 to D24, D26 to D25, D27 to D26, D28 to D27, D29 to D28, D30 to D29, D31 to D30, D32 to D31, D33 to D32, D34 to D33, D35 to D34, JP11 to JP10, JP12 to JP11, JP13 to JP12, JP14 to JP13, JP15 to JP14, JP16 to JP15, JP17 to JP16, JP18 to JP17, JP19 to JP18, JP20 to JP19, JP21 to JP20, JP22 to JP21, JP23 to JP22, JP24 to JP23, JP25 to JP24, JP26 to JP25, JP27 to JP26, JP28 to JP27, JP29 to JP28, JP30 to JP29, JP31 to JP30, JP32 to JP31, JP8 to JP7, JP9 to JP8, JP10 to JP9, R11 to R10, R12 to R11, R13 to R12, R14 to R13, R15 to R14, R16 to R15, R17 to R16, R18 to R17, R19 to R18, R20 to R19, R21 to R20, R22 to R21, R23 to R22, R24 to R23, R25 to R24, R26 to R25, R27 to R26, R28 to R27, R29 to R28, R30 to R29, R31 to R30, R32 to R31, R33 to R32, R34 to R33, R10 to R9
Connections:
- C15 pad 1: Net-(JP8-A) (its old number) -> Net-(JP7-A)
- JP7 pad 1: Net-(JP8-A) (its old number) -> Net-(JP7-A)
Routing:
- net GND: track 5.46 -> 118.6 mm, vias 4 -> 119
- net VIN 5V: track 0.00 -> 91.1 mm
- net /12V: track 0.00 -> 51.6 mm
- net /5V: track 0.00 -> 43.8 mm
- net +3V3: track 0.00 -> 21.8 mm
- net Net-(D1-K): track 0.00 -> 19.1 mm
- net /IO_23: track 0.00 -> 15.5 mm
- net /IO_19: track 0.00 -> 15.3 mm
- net /IO_22: track 0.00 -> 15.1 mm
- net /IO_18: track 0.00 -> 14.7 mm
- net /IO_11: track 0.00 -> 14.7 mm
- net /IO_12: track 0.00 -> 14.6 mm
- net Net-(Q1-S): track 0.00 -> 14.5 mm
- net /IO_5: track 0.00 -> 14.1 mm
- net /IO_17: track 0.00 -> 13.9 mm
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Other:
- board size 82 x 94.8 mm -> 78 x 94.8 mm
- board text removed: "ESP32_HEADERS"
- board text removed: "EXTERNAL CONNECTOR1"
- board text removed: "EXTERNAL CONNECTOR2"
