File: KiCad Projects/FINAL_DESIGN/FINAL_DESIGN.kicad_pcb (KiCad board)
At the start: 2 copper layers, 78 x 94.8 mm, 154 parts, among them J1 Screw_Terminal_01x02, J2 Conn_01x19_Socket, J3 Conn_01x19_Socket, J4 Conn_01x19_Socket, J5 Conn_01x19_Socket, Q1 PMOS, U1 LM2596S-5, U2 ESP32_NODEMCU

Commit message: Work:
Parts:
- moved D1 3.37 mm to (96.9, 64.2)
Routing:
- net Net-(D1-K): track 19.1 -> 21.1 mm
- net /IO_18: track 14.7 -> 13.9 mm
- net /IO_11: track 14.7 -> 14.0 mm

Commit message: work
Parts:
- moved TP2 6.25 mm to (130.5, 60.4)
Routing:
- net GND: track 118.6 -> 136.7 mm, vias 119 -> 114
- net +3V3: track 21.8 -> 17.6 mm
Changed lines of the file:
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@@
 	(footprint "TestPoint:TestPoint_Pad_D1.5mm"
 		(layer "F.Cu")
-		(at 128.675 66.375)
+		(at 130.5052 60.4012)
 		(descr "SMD pad as test Point, diameter 1.5mm")
 		(tags "test point SMD pad")
@@
 	)
 	(gr_rect
+		(start 67.35 27.3)
+		(end 145.5 27.325)
+		(stroke
+			(width 0.2)
+			(type default)
+		)
+		(fill no)
+		(layer "B.Cu")
+	)
+	(gr_rect
+		(start 67.35 27.325)
+		(end 145.5 67.25)
+		(stroke
+			(width 0.2)
+			(type default)
+		)
+		(fill no)
+		(layer "B.Cu")
+	)
+	(gr_rect
 		(start 67.575 27.475)
 		(end 145.525 122.225)
@@
 	)
 	(segment
+		(start 79.2136 75.3364)
+		(end 79.0956 75.3364)
+		(width 0.2)
+		(layer "F.Cu")
+		(net 2)
+	)
+	(segment
 		(start 128.875 107.25)
 		(end 128.725 107.4)
@@
 	)
 	(segment
-		(start 78.975 73.025)
-		(end 79.1 73.025)
-		(width 0.2)
+		(start 119.025 48.9)
+		(end 119.025 50.475)
+		(width 1)
 		(layer "F.Cu")
 		(net 2)
 	)
 	(segment
-		(start 119.025 48.9)
-		(end 119.025 50.475)
-		(width 1)
+		(start 80.7 74.775)
+		(end 79.775 74.775)
+		(width 0.2)
 		(layer "F.Cu")
 		(net 2)
@@
 	)
 	(segment
+		(start 80.75 74.25)
+		(end 81 74)
+		(width 0.2)
+		(layer "F.Cu")
+		(net 2)
+	)
+	(segment
 		(start 85.375 105.025)
 		(end 85.35 105.05)
@@
 	)
 	(segment
-		(start 84.5 68.4)
-		(end 85.125 68.4)
-		(width 0.5)
+		(start 133.8 89.075)
+		(end 134.475 88.4)
+		(width 0.2)
 		(layer "F.Cu")
 		(net 2)
 	)
 	(segment
-		(start 133.8 89.075)
-		(end 134.475 88.4)
+		(start 79.066 70.409)
+		(end 74.9302 70.409)
 		(width 0.2)
 		(layer "F.Cu")
@@
 	)
 	(segment
-		(start 80.25 75.25)
-		(end 79.775 74.775)
-		(width 0.5)
-		(layer "F.Cu")
-		(net 2)
-	)
-	(segment
 		(start 129.825 104.2)
 		(end 128.9 104.2)
@@
 	)
 	(segment
+		(start 80.75 74.825)
+		(end 80.75 74.25)
+		(width 0.2)
+		(layer "F.Cu")
+		(net 2)
+	)
+	(segment
 		(start 129.75 87.975)
 		(end 128.775 87.975)
@@
 	)
 	(segment
+		(start 79.775 74.775)
+		(end 79.2562 75.2938)
+		(width 0.2)
+		(layer "F.Cu")
+		(net 2)
+	)
+	(segment
 		(start 128.825 113.525)
 		(end 128.725 113.625)
@@
 	)
 	(segment
+		(start 80.1084 69.65)
+		(end 79.825 69.65)
+		(width 0.2)
+		(layer "F.Cu")
+		(net 2)
+	)
+	(segment
 		(start 134.45 113.85)
 		(end 134.5 113.8)
@@
 	)
 	(segment
+		(start 81.1276 68.58)
+		(end 81.1276 68.6308)
+		(width 0.2)
+		(layer "F.Cu")
+		(net 2)
+	)
+	(segment
 		(start 112.925 48.1)
 		(end 112.925 50.43976)
@@
 	)
 	(segment
+		(start 85.5 68.025)
+		(end 84.945 68.58)
+		(width 0.2)
+		(layer "F.Cu")
+		(net 2)
+	)
+	(segment
 		(start 129.8 110.55)
 		(end 128.7 110.55)
@@
 	)
 	(segment
-		(start 85.125 68.4)
-		(end 85.5 68.025)
-		(width 0.5)
-		(layer "F.Cu")
-		(net 2)
-	)
-	(segment
 		(start 134.25 78.25)
 		(end 134.25 78.325)
@@
 	)
 	(segment
+		(start 81 74)
+		(end 84.425 74)
+		(width 0.2)
+		(layer "F.Cu")
+		(net 2)
+	)
+	(segment
 		(start 85.35 114.275)
 		(end 85.325 114.3)
@@
 	)
 	(segment
+		(start 80.75 74.825)
+		(end 80.7 74.775)
+		(width 0.2)
+		(layer "F.Cu")
+		(net 2)
+	)
+	(segment
 		(start 85.375 116.175)
 		(end 85.375 117.45)
@@
 	)
 	(segment
-		(start 79.1 73.025)
-		(end 79.825 72.3)
-		(width 0.5)
-		(layer "F.Cu")
-		(net 2)
-	)
-	(segment
 		(start 93.2 40.875)
 		(end 93.15 40.825)
@@
 	)
 	(segment
-		(start 79.075 70.4)
-		(end 79.825 69.65)
+		(start 80.575 85)
+		(end 79.65 85)
 		(width 0.5)
 		(layer "F.Cu")
@@
 	)
 	(segment
-		(start 80.575 85)
-		(end 79.65 85)
-		(width 0.5)
+		(start 84.945 68.58)
+		(end 81.1276 68.58)
+		(width 0.2)
 		(layer "F.Cu")
 		(net 2)
@@
 	)
 	(segment
+		(start 79.2136 75.3364)
+		(end 74.8284 75.3364)
+		(width 0.2)
+		(layer "F.Cu")
+		(net 2)
+	)
+	(segment
+		(start 79.775 74.775)
+		(end 79.75 74.75)
+		(width 0.2)
+		(layer "F.Cu")
+		(net 2)
+	)
+	(segment
 		(start 129.725 97.725)
 		(end 128.85 97.725)
@@
 	)
 	(segment
+		(start 79.825 69.65)
+		(end 79.066 70.409)
+		(width 0.2)
+		(layer "F.Cu")
+		(net 2)
+	)
+	(segment
 		(start 134.425 99.2)
 		(end 134.425 98.5)
@@
 	)
 	(segment
-		(start 80.25 75.325)
-		(end 80.25 75.25)
+		(start 79.2562 75.2938)
+		(end 79.2136 75.3364)
 		(width 0.2)
 		(layer "F.Cu")
@@
 	)
 	(segment
-		(start 79.075 70.425)
-		(end 79.075 70.4)
-		(width 0.2)
-		(layer "F.Cu")
-		(net 2)
-	)
-	(segment
 		(start 133.9 111.925)
 		(end 133.9 111.9)
@@
 	)
 	(segment
+		(start 81.1276 68.6308)
+		(end 80.1084 69.65)
+		(width 0.2)
+		(layer "F.Cu")
+		(net 2)
+	)
+	(segment
 		(start 134.25 78.325)
 		(end 134.9 78.975)
@@
 	)
 	(via
-		(at 84.5 68.4)
-		(size 0.6)
-		(drill 0.3)
-		(layers "F.Cu" "B.Cu")
-		(free yes)
-		(net 2)
-	)
-	(via
 		(at 80.525 87.775)
 		(size 0.6)
@@
 	)
 	(via
-		(at 78.975 73.025)
-		(size 0.6)
-		(drill 0.3)
-		(layers "F.Cu" "B.Cu")
-		(free yes)
-		(net 2)
-	)
-	(via
 		(at 138.125 31.8)
 		(size 1)
@@
 	)
 	(via
-		(at 84.425 74)
-		(size 0.6)
-		(drill 0.3)
-		(layers "F.Cu" "B.Cu")
-		(free yes)
-		(net 2)
-	)
-	(via
 		(at 97.95 48.775)
 		(size 1)
@@
 	)
 	(via
-		(at 79.075 70.425)
-		(size 0.6)
-		(drill 0.3)
-		(layers "F.Cu" "B.Cu")
-		(free yes)
-		(net 2)
-	)
-	(via
 		(at 134.45 114.525)
 		(size 0.6)
@@
 	)
 	(via
-		(at 80.25 75.325)
-		(size 0.6)
-		(drill 0.3)
-		(layers "F.Cu" "B.Cu")
-		(free yes)
-		(net 2)
-	)
-	(via
 		(at 119.025 48.9)
 		(size 1)
@@
 	)
 	(segment
-		(start 131.5 69.2)
-		(end 131.5 69.415)
-		(width 0.2)
-		(layer "F.Cu")
-		(net 133)
-	)
-	(segment
 		(start 131.5 69.415)
 		(end 136.62 69.415)
@@
 		(width 0.5)
 		(layer "F.Cu")
-		(net 133)
-	)
-	(segment
-		(start 128.675 66.375)
-		(end 131.5 69.2)
-		(width 0.5)
-		(layer "F.Cu")
