File: KiCad Projects/ESP_32 DESIGN/ESP_32/_autosave-untitled.kicad_sch (KiCad schematic)
At the start: 147 parts, among them J1 Screw_Terminal_01x02, J2 Conn_01x19_Socket, J3 Conn_01x19_Socket, J4 Conn_01x19_Socket, J5 Conn_01x19_Socket, Q1 PMOS, U1 LM2596S-5, U2 ESP32_NODEMCU

Commit message: work
Other:
- company: KCT -> (none)
- title: ESP32 CARRIER BOARD -> (none)
- moved on the sheet: C1, C10, C11, C12, C13, C14, C16, C17, C18, C19, C2, C20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
