File: KiCad Projects/ESP_32 DESIGN/ESP_32/ESP_32.kicad_sch (KiCad schematic)
At the start: 27 parts, among them J11 Screw_Terminal_01x02, J12 Conn_01x19_Socket, J13 Conn_01x19_Socket, J14 Conn_01x19_Socket, J15 Conn_01x19_Socket, Q3 PMOS, U5 LM2596S-5, U6 ESP32_NODEMCU

Commit message: stm & pcb
Parts:
- removed C49: 680uF, Capacitor_THT:CP_Radial_D6.3mm_P2.50mm, symbol Device:C_Polarized
- removed C50, C53: 220uF, Capacitor_THT:CP_Radial_D6.3mm_P2.50mm, symbol Device:C_Polarized
- removed C51: 470uF, Capacitor_THT:CP_Radial_D6.3mm_P2.50mm, symbol Device:C_Polarized
- removed C52, C55: 10uF, Capacitor_THT:C_Disc_D3.0mm_W2.0mm_P2.50mm, symbol Device:C
- removed C54, C56: 0.1uF, Capacitor_THT:C_Disc_D3.0mm_W1.6mm_P2.50mm, symbol Device:C
- removed C57: 100nf, Capacitor_SMD:C_0805_2012Metric, symbol Device:C
- removed D39: 1N5824, Diode_SMD:D_01005_0402Metric_Pad0.57x0.30mm_HandSolder, symbol Device:D
- removed D40: D_Zener, Diode_THT:D_5W_P10.16mm_Horizontal, symbol Device:D_Zener
- removed D41: Shottky, Diode_THT:D_DO-201_P15.24mm_Horizontal, symbol Device:D
- removed D42: D_Zener, Diode_SMD:D_SOD-882, symbol Device:D_Zener
- removed F3: 3A, Fuse:FuseHolder_Blade_ATO_Littelfuse_FLR_178.6165, symbol Device:Polyfuse
- removed J11: Screw_Terminal_01x02, TerminalBlock_4Ucon:TerminalBlock_4Ucon_1x02_P3.50mm_Vertical, symbol Connector:Screw_Terminal_01x02
- removed JP33: SolderJumper_2_Open, Jumper:SolderJumper-2_P1.3mm_Open_Pad1.0x1.5mm, symbol Jumper:SolderJumper_2_Open
- removed L3: WE-PD2_4532, Inductor_SMD:L_Wuerth_WE-PD2-Typ-MS, symbol WE-PD2_4532:WE-PD2_4532
- removed Q3: PMOS, Package_TO_SOT_THT:TO-92L_HandSolder, symbol Simulation_SPICE:PMOS
- removed R37, R38: 100K, Resistor_SMD:R_0805_2012Metric_Pad1.20x1.40mm_HandSolder, symbol Device:R
- removed R39: 150, Resistor_SMD:R_0805_2012Metric, symbol RC0805FR-07330RL:RC0805FR-07330RL
- removed U5: LM2596S-5, Package_TO_SOT_SMD:TO-263-5_TabPin3, symbol Regulator_Switching:LM2596S-5
- removed U6: ESP32_NODEMCU, MODULE_ESP32_NODEMCU, symbol ESP32_NODEMCU:ESP32_NODEMCU
Other:
- note removed: "ESP32"
- note removed: "Note: All Capcitors 10V"
- note removed: "Note: All Capcitors 25V"
- note removed: "Power Circuit"
