File: KiCad Projects/ESP32_PCB_ONLY_PINS/FINAL_DESIGN.kicad_pcb (KiCad board)
At the start: 2 copper layers, 78 x 94.8 mm, 154 parts, among them J1 Screw_Terminal_01x02, J2 Conn_01x19_Socket, J3 Conn_01x19_Socket, J4 Conn_01x19_Socket, J5 Conn_01x19_Socket, Q1 PMOS, U1 LM2596S-5, U2 ESP32_NODEMCU

Commit message: pcb
Parts:
- removed C10, C11, C12, C13, C14, C15 (x2), C16, C17, C18, C19, C20, C21, C22, C23, C24, C25, C26, C27, C28, C29, C30, C31, C32, C33, C34, C35, C36, C37, C38, C39, C9: 100nf, Capacitor_SMD:C_0805_2012Metric
- removed the D10 at (79.8, 69.3)
- removed the D10 at (79.8, 72.0)
- removed D25, D26, D27, D28, D29, D30, D31, D32, D33, D34: D_Zener, Diode_SMD:D_SOD-882
- removed JP1, JP10, JP11, JP12, JP13, JP14, JP15, JP16, JP17, JP18, JP19, JP2, JP20, JP21, JP22, JP23, JP24, JP25, JP26, JP27, JP28, JP29, JP3, JP30, JP31, JP4, JP5, JP6, JP7 (x2), JP8, JP9: SolderJumper_2_Open, Jumper:SolderJumper-2_P1.3mm_Open_Pad1.0x1.5mm
- removed R24, R25, R26, R27, R28, R29, R30, R31, R32, R33: 150, RC0805FR-07330RL:RESC2012X60N
- removed the R9 at (82.7, 67.2)
- removed the R9 at (82.7, 69.8)
- added D10: D_Zener, Diode_SMD:D_SOD-882, F.Cu at (87.0, 94.3)
- added R9: 100, RC0805FR-07330RL:RESC2012X60N, F.Cu at (90.5, 94.3)
- R10, R11, R12, R13, R14, R15, R16, R17, R18, R19, R20, R21, R22, R23, R5, R6, R7, R8: value 150 -> 100
- R3, R4: value 150 -> 33
- moved D24 57.9 mm to (130.2, 81.7), turned to 0 degrees
- moved D23 55.4 mm to (129.8, 78.8), turned to 0 degrees
- moved D18 53.6 mm to (128.6, 99.0), turned to 0 degrees
- moved D8 52.1 mm to (128.6, 102.4), turned to 0 degrees
- moved D21 51.9 mm to (130.3, 83.8), turned to 0 degrees
- moved D22 51.1 mm to (129.6, 86.5), turned to 0 degrees
- moved D15 50.8 mm to (86.5, 118.0), turned to 0 degrees
- moved D20 50.4 mm to (129.9, 91.4), turned to 0 degrees
- moved D19 49.9 mm to (129.5, 89.0), turned to 0 degrees
- moved R23 49.7 mm to (122.4, 81.6)
- moved D7 49.4 mm to (128.9, 109.6), turned to 0 degrees
- moved D13 47.9 mm to (86.8, 106.7), turned to 0 degrees
- moved D12 47.7 mm to (87.2, 101.9), turned to 0 degrees
- moved D14 47.7 mm to (86.8, 115.0), turned to 0 degrees
- moved D16 47.5 mm to (86.9, 104.7), turned to 0 degrees
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Connections:
- D11 pad 1: /SD1 -> /I/O_18
- D12 pad 1: /SD2 -> /I/O_19
- D13 pad 1: /SD3 -> /I/O_21
- D14 pad 1: /CMD -> /I/O_22
- D15 pad 1: /I/O_12 -> /I/O_23
- D16 pad 1: /I/O_13 -> /I/O_25
- D17 pad 1: /I/O_14 -> /I/O_26
- D18 pad 1: /I/O_15 -> /I/O_27
- D19 pad 1: /I/O_16 -> /I/O_32
- D20 pad 1: /I/O_17 -> /I/O_33
- D21 pad 1: /I/O_18 -> /I/O_34
- D22 pad 1: /I/O_19 -> /I/O_35
- D23 pad 1: /I/O_21 -> /SP
- D24 pad 1: /I/O_22 -> /SN
- D4 pad 1: /I/O_0 -> /TXD
- D5 pad 1: /TXD -> /RXD
- D6 pad 1: /I/O_2 -> /I/O_4
- D7 pad 1: /RXD -> /I/O_13
- D8 pad 1: /I/O_4 -> /I/O_14
- D9 pad 1: /I/O_5 -> /I/O_16
- R10 pad 1: /SD1 -> /I/O_18
- R10 pad 2: /IO_8 -> /IO_18
- R11 pad 1: /SD2 -> /I/O_19
- R11 pad 2: /IO_9 -> /IO_19
- R12 pad 1: /SD3 -> /I/O_21
- R12 pad 2: /IO_10 -> /IO_21
- R13 pad 1: /CMD -> /I/O_22
- R13 pad 2: /IO_11 -> /IO_22
- R14 pad 1: /I/O_12 -> /I/O_23
- R14 pad 2: /IO_12 -> /IO_23
- R15 pad 1: /I/O_13 -> /I/O_25
- R15 pad 2: /IO_13 -> /IO_25
- R16 pad 1: /I/O_14 -> /I/O_26
- R16 pad 2: /IO_14 -> /IO_26
- R17 pad 1: /I/O_15 -> /I/O_27
- R17 pad 2: /IO_15 -> /IO_27
- R18 pad 1: /I/O_16 -> /I/O_32
- R18 pad 2: /IO16 -> /IO_32
- R19 pad 1: /I/O_17 -> /I/O_33
- R19 pad 2: /IO_17 -> /IO_33
- R20 pad 1: /I/O_18 -> /I/O_34
- R20 pad 2: /IO_18 -> /IO_34
- R21 pad 1: /I/O_19 -> /I/O_35
- R21 pad 2: /IO_19 -> /IO_35
- R22 pad 1: /I/O_21 -> /SP
- R22 pad 2: /IO_21 -> /IO_36
- R23 pad 1: /I/O_22 -> /SN
- R23 pad 2: /IO_22 -> /IO_39
- R3 pad 1: /I/O_0 -> /TXD
- R3 pad 2: /IO_0 -> /IO_1
- R4 pad 1: /TXD -> /RXD
- R4 pad 2: /IO_1 -> /IO_3
- R5 pad 1: /I/O_2 -> /I/O_4
- R5 pad 2: /IO_2 -> /IO_4
- R6 pad 1: /RXD -> /I/O_13
- R6 pad 2: /IO_3 -> /IO_13
- R7 pad 1: /I/O_4 -> /I/O_14
- R7 pad 2: /IO_4 -> /IO_14
- R8 pad 1: /I/O_5 -> /I/O_16
- R8 pad 2: /IO_5 -> /IO16
Routing:
- net GND: track 136.7 -> 50.5 mm, vias 114 -> 56
- net VIN 5V: track 91.1 -> 63.5 mm
- net +3V3: track 17.6 -> 0.00 mm
- net /IO_23: track 15.5 -> 0.00 mm
- net /IO_19: track 15.3 -> 0.00 mm
- net /IO_22: track 15.1 -> 0.00 mm
- net /IO_1: track 14.4 -> 0.00 mm
- net /IO_11: track 14.0 -> 0.00 mm
- net /IO_18: track 13.9 -> 0.00 mm
- net /IO_3: track 13.9 -> 0.00 mm
- net /IO_5: track 13.9 -> 0.00 mm
- net /IO_17: track 13.9 -> 0.00 mm
- net /IO_21: track 13.8 -> 0.00 mm
- net /IO_10: track 13.7 -> 0.00 mm
- net /IO_14: track 13.7 -> 0.00 mm
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
Commit message: PCB MODIFIED INSIDE ONLYPINS
Parts:
- removed D23, D24: D_Zener, Diode_SMD:D_SOD-882
- removed J3, J5: Conn_01x19_Socket, Connector_PinHeader_2.54mm:PinHeader_1x19_P2.54mm_Vertical
- removed R22, R23: 100, RC0805FR-07330RL:RESC2012X60N
- added J6: TB010-508-P19BK, TB010-508-P19BK:CUI_TB010-508-P19BK, F.Cu at (163.2, 69.9)
- added J7: TB010-508-P19BK, TB010-508-P19BK:CUI_TB010-508-P19BK, F.Cu at (70.6, 70.1)
- moved D16 69.4 mm to (155.9, 112.3), turned to 180 degrees
- moved U2 58.3 mm to (236.2, 106.2)
- moved R15 44.6 mm to (133.5, 137.1), turned to 180 degrees
- moved R7 44.5 mm to (133.5, 145.5), turned to 180 degrees
- moved R21 44.5 mm to (133.5, 129.5), turned to 180 degrees
- moved J4 44.4 mm to (129.6, 116.8)
- moved R17 44.4 mm to (133.6, 142.3), turned to 180 degrees
- moved R16 44.3 mm to (133.6, 139.7), turned to 180 degrees
- moved R19 44.3 mm to (133.5, 134.4), turned to 180 degrees
- moved R18 44.3 mm to (133.5, 132.0), turned to 180 degrees
- moved R20 44.3 mm to (133.5, 127.0), turned to 180 degrees
- moved R12 44.1 mm to (99.7, 149.5)
- moved R14 44.1 mm to (99.7, 160.5)
- moved R3 44.1 mm to (99.7, 155.0)
- moved R4 44.0 mm to (99.7, 152.3)
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Connections:
- J2 pad 1: /IO_6 -> /CLK
- J2 pad 10: /IO_5 -> /I/O_5
- J2 pad 2: /IO_7 -> /SD0
- J2 pad 3: /IO_8 -> /SD1
- J2 pad 4: /IO_15 -> /I/O_15
- J2 pad 5: /IO_2 -> /I/O_2
- J2 pad 6: /IO_0 -> /I/O_0
- J4 pad 13: /IO_12 -> /I/O_12
- J4 pad 16: /IO_9 -> /SD2
- J4 pad 17: /IO_10 -> /SD3
- J4 pad 18: /IO_11 -> /CMD
- J4 pad 3: /IO_36 -> /SP
- J4 pad 4: /IO_39 -> /SN
- R8 pad 2: /IO16 -> /IO_16
Routing:
- net GND: track 50.5 -> 164.2 mm, vias 56 -> 0
- net VIN 5V: track 63.5 -> 159.1 mm
- net +3V3: track 0.00 -> 66.7 mm
- net /CLK: track 0.00 -> 60.8 mm
- net /EN: track 0.00 -> 59.3 mm
- net /SD0: track 0.00 -> 58.3 mm
- net /SD1: track 0.00 -> 55.8 mm
- net /SP: track 0.00 -> 55.7 mm
- net /SN: track 0.00 -> 54.6 mm
- net /I/O_15: track 0.00 -> 53.2 mm
- net /I/O_35: track 0.00 -> 50.9 mm
- net /I/O_2: track 0.00 -> 50.7 mm
- net /I/O_0: track 0.00 -> 49.5 mm
- net /I/O_32: track 0.00 -> 47.8 mm
- net /I/O_33: track 0.00 -> 45.2 mm
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- added copper zone on F.Cu, net GND
- removed copper zone on B.Cu, net GND
Other:
- board size 78 x 94.8 mm -> 113.4 x 132.9 mm

Commit message: PCB CHANGE
Parts:
- moved U2 36.9 mm to (208.5, 130.5)
- moved F1 11.9 mm to (150.4, 49.2)
- moved J1 11.2 mm to (160.1, 47.3)
- moved D16 9.41 mm to (146.5, 112.3)
- moved D21 9.12 mm to (146.5, 91.0)
- moved D8 9.05 mm to (146.5, 125.9)
- moved D22 9.04 mm to (146.5, 95.5)
- moved D18 9.03 mm to (146.5, 120.7)
- moved D19 9.02 mm to (146.5, 100.5)
- moved D17 8.97 mm to (146.5, 117.9)
- moved D7 8.96 mm to (146.5, 141.3)
- moved D20 8.94 mm to (146.5, 105.4)
- moved J6 8.69 mm to (154.5, 69.9)
- moved D15 8.66 mm to (87.0, 156.5)
- moved D14 8.55 mm to (87.0, 151.3)
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Routing:
- net GND: track 164.2 -> 33.8 mm
- net /I/O_34: track 0.07 -> 49.0 mm
- net VIN 5V: track 159.1 -> 114.7 mm
- net /I/O_12: track 0.00 -> 31.8 mm
- net /I/O_21: track 35.1 -> 26.3 mm
- net /I/O_13: track 33.6 -> 24.9 mm
- net /RXD: track 33.3 -> 24.7 mm
- net /SD2: track 37.2 -> 28.6 mm
- net /CMD: track 35.1 -> 26.5 mm
- net /SD3: track 36.2 -> 27.6 mm
- net Net-(Q1-S): track 14.5 -> 23.1 mm
- net /TXD: track 32.3 -> 23.8 mm
- net /I/O_22: track 31.2 -> 22.7 mm
- net /I/O_23: track 30.1 -> 21.8 mm
- net Net-(J1-Pin_1): track 10.6 -> 18.4 mm
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Other:
- board size 113.4 x 132.9 mm -> 98.2 x 126.9 mm
