File: KiCad Projects/ESP32_PCB_ONLY_PINS/FINAL_DESIGN.kicad_pcb (KiCad board)
At the start: 2 copper layers, 98.2 x 126.9 mm, 64 parts, among them J1 Screw_Terminal_01x02, J2 Conn_01x19_Socket, J4 Conn_01x19_Socket, J6 TB010-508-P19BK, J7 TB010-508-P19BK, Q1 PMOS, U1 LM2596S-5, U2 ESP32_NODEMCU

Commit message: FINAL PCB WORK
Parts:
- added G***: LOGO, QBOTIX_LOGO:QBOTIX_LOGO, F.Cu at (118.6, 94.0)
- added G***: LOGO, LOGO:LOGO, F.Cu at (208.5, 115.8)
- added G***: LOGO, ROBOCON2026_LOGO:ROBOCON 2026 LOGO, F.Cu at (116.6, 37.5)
- added REF**: MountingHole_2.2mm_M2, MountingHole:MountingHole_2.2mm_M2, F.Cu at (70.5, 37.2)
- added REF**: MountingHole_2.2mm_M2, MountingHole:MountingHole_2.2mm_M2, F.Cu at (163.4, 37.2)
- added REF**: MountingHole_2.2mm_M2, MountingHole:MountingHole_2.2mm_M2, F.Cu at (163.4, 166.6)
- added REF**: MountingHole_2.2mm_M2, MountingHole:MountingHole_2.2mm_M2, F.Cu at (70.5, 166.7)
- D1: footprint Diode_SMD:D_01005_0402Metric_Pad0.57x0.30mm_HandSolder -> 1N5824:DIOAD1898W129L762D1143
- moved D1 11.2 mm to (114.9, 80.5), turned to 0 degrees
- moved R1 3.19 mm to (126.3, 46.0)
- moved R2 1.96 mm to (121.0, 44.1), turned to 90 degrees
- moved D18 0.50 mm to (146.8, 121.1)
- moved D19 0.26 mm to (146.7, 100.5)
- renumbered J7 to J2, J2 to J3, J6 to J4, J4 to J5
Connections:
- L1 pad 1: Net-(D1-K) -> Net-(U1-OUT)
- U1 pad 2: Net-(D1-K) -> Net-(U1-OUT)
Routing:
- net Net-(U1-OUT): track 0.00 -> 27.7 mm
- net VIN 5V: track 114.7 -> 140.2 mm
- net Net-(D1-K): track 21.1 -> 0.00 mm
- net Net-(Q1-S): track 23.1 -> 39.3 mm
- net GND: track 33.8 -> 43.9 mm
- net Net-(Q1-G): track 7.62 -> 11.6 mm
- net /I/O_27: track 34.6 -> 35.5 mm
Other:
- board size 98.2 x 126.9 mm -> 100.9 x 137.5 mm

Commit message: changes
Parts:
- removed the G*** at (208.5, 115.8)
- removed U2: ESP32_NODEMCU, ESP32_NODEMCU:MODULE_ESP32_NODEMCU
- moved R5 0.20 mm to (99.7, 129.6)
- moved D20 0.20 mm to (146.4, 105.2)
- moved L1 0.20 mm to (113.5, 68.7)
- moved C1 0.20 mm to (91.6, 52.8)
- moved R2 0.20 mm to (120.9, 43.9)
- moved REF** 0.20 mm to (70.5, 37.0)
- moved REF** 0.20 mm to (163.3, 37.0)
- moved TP1 0.20 mm to (114.7, 52.6)
- moved C2 0.20 mm to (115.4, 61.2)
- moved C3 0.20 mm to (103.0, 43.8)
- moved C5 0.20 mm to (122.8, 61.1)
- moved C6 0.20 mm to (97.3, 44.0)
- moved C7 0.20 mm to (131.9, 61.2)
- moved C8 0.20 mm to (128.9, 61.2)
- moved D1 0.20 mm to (114.8, 80.3)
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
Commit message: PCB FINAL WORK DONE
Parts:
- removed D10, D11, D12, D13, D14, D15, D16, D17, D18, D19, D20, D21, D22, D4, D5, D6, D7, D8, D9: D_Zener, Diode_SMD:D_SOD-882
- removed D3: Shottky, Diode_THT:D_DO-201_P15.24mm_Horizontal
- added CR1: PESD3V3L1BA_115, footprints:DIODE_PESD3V3L1BA_115_NEX, F.Cu at (88.9, 147.3)
- added CR10: PESD3V3L1BA_115, footprints:DIODE_PESD3V3L1BA_115_NEX, F.Cu at (88.9, 136.9)
- added CR11: PESD3V3L1BA_115, footprints:DIODE_PESD3V3L1BA_115_NEX, F.Cu at (88.9, 152.1)
- added CR12: PESD3V3L1BA_115, footprints:DIODE_PESD3V3L1BA_115_NEX, F.Cu at (88.9, 161.5)
- added CR13: PESD3V3L1BA_115, footprints:DIODE_PESD3V3L1BA_115_NEX, F.Cu at (144.4, 111.8)
- added CR14: PESD3V3L1BA_115, footprints:DIODE_PESD3V3L1BA_115_NEX, F.Cu at (144.4, 116.6)
- added CR15: PESD3V3L1BA_115, footprints:DIODE_PESD3V3L1BA_115_NEX, F.Cu at (144.4, 121.9)
- added CR16: PESD3V3L1BA_115, footprints:DIODE_PESD3V3L1BA_115_NEX, F.Cu at (144.4, 102.1)
- added CR17: PESD3V3L1BA_115, footprints:DIODE_PESD3V3L1BA_115_NEX, F.Cu at (144.4, 106.7)
- added CR18: PESD3V3L1BA_115, footprints:DIODE_PESD3V3L1BA_115_NEX, F.Cu at (144.4, 93.0)
- added CR19: PESD3V3L1BA_115, footprints:DIODE_PESD3V3L1BA_115_NEX, F.Cu at (144.4, 97.5)
- added CR2: PESD3V3L1BA_115, footprints:DIODE_PESD3V3L1BA_115_NEX, F.Cu at (88.9, 142.2)
- added CR3: PESD3V3L1BA_115, footprints:DIODE_PESD3V3L1BA_115_NEX, F.Cu at (88.9, 105.9)
- added CR4: PESD3V3L1BA_115, footprints:DIODE_PESD3V3L1BA_115_NEX, F.Cu at (144.5, 144.3)
- added CR5: PESD3V3L1BA_115, footprints:DIODE_PESD3V3L1BA_115_NEX, F.Cu at (144.4, 127.0)
- added CR6: PESD3V3L1BA_115, footprints:DIODE_PESD3V3L1BA_115_NEX, F.Cu at (88.9, 110.5)
- added CR7: PESD3V3L1BA_115, footprints:DIODE_PESD3V3L1BA_115_NEX, F.Cu at (88.9, 115.3)
- added CR8: PESD3V3L1BA_115, footprints:DIODE_PESD3V3L1BA_115_NEX, F.Cu at (88.9, 125.7)
- added CR9: PESD3V3L1BA_115, footprints:DIODE_PESD3V3L1BA_115_NEX, F.Cu at (88.9, 130.8)
- C1: footprint Capacitor_THT:CP_Radial_D6.3mm_P2.50mm -> Capacitor_THT:CP_Radial_D10.0mm_P5.00mm
- C3: footprint Capacitor_THT:CP_Radial_D6.3mm_P2.50mm -> Capacitor_THT:CP_Radial_D8.0mm_P3.50mm
- C4, C7: footprint Capacitor_THT:C_Disc_D3.0mm_W2.0mm_P2.50mm -> Capacitor_SMD:C_0805_2012Metric
- C6, C8: footprint Capacitor_THT:C_Disc_D3.0mm_W1.6mm_P2.50mm -> Capacitor_SMD:C_0805_2012Metric
- D1: value 1N5824 -> SS34; footprint 1N5824:DIOAD1898W129L762D1143 -> SS34:DIO_SS34
- D2: value D_Zener -> MMBZ5242B-7-F; footprint Diode_THT:D_5W_P10.16mm_Horizontal -> MMBZ5242B-7-F:SOT91P240X102-3N
- J1: footprint TerminalBlock_4Ucon:TerminalBlock_4Ucon_1x02_P3.50mm_Vertical -> Connector_Phoenix_MC_HighVoltage:PhoenixContact_MCV_1,5_2-G-5.08_1x02_P5.08mm_Vertical
- Q1: value PMOS -> AO3401A; footprint Package_TO_SOT_THT:TO-92L_HandSolder -> A03401:SOT23-3
- R10, R11, R12, R13, R14, R15, R16, R17, R18, R19, R20, R21, R3, R4, R5, R6, R7, R8, R9: footprint RC0805FR-07330RL:RESC2012X60N -> Resistor_SMD:R_0805_2012Metric
- TP1 +12V: renamed from TP1
- TP2 +3V3: renamed from TP2
- TP3 +5V5: renamed from TP3
- moved TP3 +5V5 14.5 mm to (138.3, 61.1)
- moved D1 13.9 mm to (126.6, 72.9)
- moved J1 3.97 mm to (161.5, 50.8)
- moved L1 3.03 mm to (115.5, 71.1)
- moved R2 2.85 mm to (120.9, 46.7), turned to -90 degrees
- moved D2 2.17 mm to (111.3, 46.0), turned to 0 degrees
- moved Q1 2.12 mm to (115.1, 45.0)
- moved R1 1.19 mm to (125.2, 45.2), turned to -90 degrees
- moved C7 1.08 mm to (132.1, 60.1)
- moved C8 1.08 mm to (129.1, 60.1)
- moved R11 1.05 mm to (100.4, 143.3)
- moved R10 0.89 mm to (99.9, 140.5)
- moved R9 0.75 mm to (100.3, 135.4)
- moved R5 0.64 mm to (100.3, 129.4)
- moved R20 0.29 mm to (133.4, 126.8)
Connections:
- C2 pad 1: /5V -> VIN 5V
- C5 pad 1: /5V -> VIN 5V
- C7 pad 1: /5V -> VIN 5V
- C8 pad 1: /5V -> VIN 5V
- D2 pad 1: /12V -> GND
- D2 pad 2: GND -> (no net)
- F1 pad 2: Net-(Q1-S) -> Net-(F1-Pad2)
- L1 pad 2: /5V -> VIN 5V
- Q1 pad 1: /12V -> Net-(Q1-Pad1)
- Q1 pad 2: Net-(Q1-G) -> Net-(F1-Pad2)
- Q1 pad 3: Net-(Q1-S) -> /12V
- R1 pad 1: Net-(Q1-S) -> Net-(F1-Pad2)
- R1 pad 2: Net-(Q1-G) -> Net-(Q1-Pad1)
- R2 pad 1: Net-(Q1-G) -> Net-(Q1-Pad1)
- U1 pad 4: /5V -> VIN 5V
Routing:
- net VIN 5V: track 140.2 -> 201.6 mm
- net /5V: track 43.8 -> 0.00 mm
- net Net-(Q1-S): track 39.3 -> 0.00 mm
- net Net-(F1-Pad2): track 0.00 -> 31.4 mm
- net Net-(Q1-G): track 11.6 -> 0.00 mm
- net Net-(Q1-Pad1): track 0.00 -> 9.43 mm
- net GND: track 43.9 -> 35.1 mm
- net /I/O_5: track 43.0 -> 39.6 mm
- net /I/O_26: track 35.5 -> 38.4 mm
- net /I/O_25: track 38.2 -> 40.6 mm
- net /12V: track 51.6 -> 53.9 mm
- net Net-(J1-Pin_1): track 18.4 -> 20.4 mm
- net /I/O_18: track 33.5 -> 31.9 mm
- net /I/O_21: track 26.3 -> 27.9 mm
- net /I/O_33: track 41.7 -> 43.0 mm
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Other:
- board size 100.9 x 137.5 mm -> 101.4 x 138.9 mm

Commit message: wr
Parts:
- C4, C6, C7, C8: footprint Capacitor_SMD:C_0805_2012Metric -> Capacitor_SMD:C_1206_3216Metric
- R1, R2: footprint Resistor_SMD:R_0805_2012Metric_Pad1.20x1.40mm_HandSolder -> Resistor_SMD:R_1206_3216Metric
- R10, R11, R12, R13, R14, R15, R16, R17, R18, R19, R20, R21, R3, R4, R5, R6, R7, R8, R9: footprint Resistor_SMD:R_0805_2012Metric -> Resistor_SMD:R_1206_3216Metric
- TP1: renamed from TP1 +12V
- TP2: renamed from TP2 +3V3
- TP3: renamed from TP3 +5V5
- moved R20 1.49 mm to (134.9, 126.8)
- moved R6 1.44 mm to (134.9, 152.0)
- moved R15 1.21 mm to (134.9, 136.9)
- moved R16 1.21 mm to (134.9, 139.5)
- moved R17 1.21 mm to (134.9, 142.2)
- moved R18 1.21 mm to (134.9, 131.8)
- moved R19 1.21 mm to (134.9, 134.2)
- moved R21 1.21 mm to (134.9, 129.3)
- moved R7 1.21 mm to (134.9, 145.3)
- moved CR4 0.11 mm to (144.4, 144.3)
- renumbered REF** to H1, REF** to H2, REF** to H3, REF** to H4
Connections:
- net /CLK renamed CLK
- net /CMD renamed CMD
- net /EN renamed EN
- net /IO_1 renamed IO_1
- net /IO_13 renamed IO_13
- net /IO_14 renamed IO_14
- net /IO_16 renamed IO_16
- net /IO_17 renamed IO_17
- net /IO_18 renamed IO_18
- net /IO_19 renamed IO_19
- net /IO_21 renamed IO_21
- net /IO_22 renamed IO_22
- net /IO_23 renamed IO_23
- net /IO_25 renamed IO_25
- net /IO_26 renamed IO_26
- net /IO_27 renamed IO_27
- net /IO_3 renamed IO_3
- net /IO_32 renamed IO_32
- net /IO_33 renamed IO_33
- net /IO_34 renamed IO_34
- net /IO_35 renamed IO_35
- net /IO_4 renamed IO_4
- net /I/O_0 renamed I/O_0
- net /I/O_12 renamed I/O_12
- net /I/O_13 renamed I/O_13
- net /I/O_14 renamed I/O_14
- net /I/O_15 renamed I/O_15
- net /I/O_16 renamed I/O_16
- net /I/O_17 renamed I/O_17
- net /I/O_18 renamed I/O_18
- net /I/O_19 renamed I/O_19
- net /I/O_2 renamed I/O_2
- net /I/O_21 renamed I/O_21
- net /I/O_22 renamed I/O_22
- net /I/O_23 renamed I/O_23
- net /I/O_25 renamed I/O_25
- net /I/O_26 renamed I/O_26
- net /I/O_27 renamed I/O_27
- net /I/O_32 renamed I/O_32
- net /I/O_33 renamed I/O_33
- net /I/O_34 renamed I/O_34
- net /I/O_35 renamed I/O_35
- net /I/O_4 renamed I/O_4
- net /I/O_5 renamed I/O_5
- net /RXD renamed RXD
- net /SD0 renamed SD0
- net /SD1 renamed SD1
- net /SD2 renamed SD2
- net /SD3 renamed SD3
- net /SN renamed SN
- net /SP renamed SP
- net /TXD renamed TXD
Routing:
- net I/O_35: track 47.6 -> 0.00 mm
- net I/O_32: track 45.3 -> 0.90 mm
- net I/O_12: track 31.8 -> 0.00 mm
- net SD2: track 28.6 -> 0.00 mm
- net SD3: track 27.6 -> 0.00 mm
- net CMD: track 26.5 -> 0.00 mm
- net I/O_14: track 33.7 -> 22.9 mm
- net I/O_27: track 35.6 -> 24.9 mm
- net I/O_26: track 38.4 -> 27.8 mm
- net I/O_33: track 43.0 -> 32.4 mm
- net I/O_25: track 40.6 -> 30.0 mm
- net EN: track 54.7 -> 64.3 mm
- net SP: track 53.2 -> 61.9 mm
- net +3V3: track 62.3 -> 65.8 mm
- net IO_25: track 3.34 -> 0.01 mm
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- removed copper zone on F.Cu, net GND
Other:
- board text added: "REV 0.00"

Commit message: work
Parts:
- moved CR5 10.1 mm to (145.5, 137.0)
- moved CR11 6.85 mm to (88.9, 159.0)
- moved CR15 6.66 mm to (145.4, 128.5)
- moved CR14 6.01 mm to (145.5, 122.5)
- moved CR1 5.68 mm to (88.9, 153.0)
- moved CR2 5.26 mm to (88.9, 147.5)
- moved CR10 4.59 mm to (89.0, 141.5)
- moved CR13 4.36 mm to (145.4, 116.0)
- moved CR9 4.19 mm to (89.0, 135.0)
- moved CR12 3.50 mm to (88.9, 165.0)
- moved CR7 3.18 mm to (88.9, 118.5)
- moved CR17 2.99 mm to (145.4, 109.5)
- moved CR8 2.77 mm to (88.9, 128.5)
- moved R11 2.71 mm to (98.5, 145.3)
- moved R9 2.68 mm to (98.5, 137.4)
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Routing:
- net I/O_35: track 0.00 -> 39.6 mm
- net I/O_12: track 0.00 -> 32.9 mm
- net SD2: track 0.00 -> 28.6 mm
- net SD3: track 0.00 -> 27.6 mm
- net CMD: track 0.00 -> 26.5 mm
- net I/O_33: track 32.4 -> 43.4 mm
- net GND: track 35.1 -> 24.4 mm
- net CLK: track 57.2 -> 67.9 mm
- net I/O_34: track 51.5 -> 41.4 mm
- net SD1: track 52.1 -> 61.9 mm
- net I/O_25: track 30.0 -> 39.3 mm
- net I/O_15: track 49.6 -> 58.2 mm
- net SD0: track 54.7 -> 63.0 mm
- net I/O_26: track 27.8 -> 36.0 mm
- net I/O_27: track 24.9 -> 32.3 mm
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- added copper zone on F.Cu, net GND

Commit message: work
Parts:
- F1: value 3A -> 4628; footprint Fuse:FuseHolder_Blade_ATO_Littelfuse_FLR_178.6165 -> CATRIDGE_FUSE:FUSE_4628
- moved C6 13.4 mm to (83.9, 44.6)
- moved C1 13.1 mm to (78.9, 49.5)
- moved C8 11.6 mm to (140.7, 59.7)
- moved F1 8.91 mm to (141.5, 48.1)
- moved TP3 8.60 mm to (146.9, 61.2)
- moved TP1 6.09 mm to (120.7, 53.9)
- moved CR15 6.05 mm to (145.4, 134.6)
- moved C4 5.73 mm to (89.0, 44.6)
- moved C3 5.46 mm to (97.6, 43.1)
- moved C5 4.62 mm to (127.4, 61.2)
- moved C7 3.69 mm to (135.8, 59.7)
- moved R20 3.53 mm to (134.7, 123.2)
- moved R8 3.22 mm to (98.4, 131.5)
- moved R5 3.10 mm to (98.4, 128.2)
- moved CR4 2.73 mm to (145.4, 148.2)
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Routing:
- net I/O_32: track 2.74 -> 44.2 mm
- net /12V: track 53.9 -> 83.0 mm
- net Net-(F1-Pad2): track 31.4 -> 16.2 mm
- net Net-(J1-Pin_1): track 20.4 -> 9.89 mm
- net GND: track 24.4 -> 16.1 mm
- net SD0: track 63.0 -> 54.9 mm
- net SD1: track 61.9 -> 54.4 mm
- net I/O_35: track 39.6 -> 46.7 mm
- net I/O_0: track 52.6 -> 45.8 mm
- net I/O_4: track 44.8 -> 39.1 mm
- net I/O_34: track 41.4 -> 47.0 mm
- net I/O_16: track 43.6 -> 38.3 mm
- net I/O_5: track 43.0 -> 38.0 mm
- net I/O_17: track 39.5 -> 35.2 mm
- net I/O_2: track 54.3 -> 50.0 mm
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