File: KiCad Projects/ESP32_PCB_ONLY_PINS/FINAL_DESIGN.kicad_sch (KiCad schematic)
At the start: 68 parts, among them J1 Screw_Terminal_01x02, J2 Conn_01x19_Socket, J3 Conn_01x19_Socket, J4 Conn_01x19_Socket, J5 Conn_01x19_Socket, Q1 PMOS, U1 LM2596S-5, U2 ESP32_NODEMCU

Commit message: pcb
Parts:
- renumbered D20 to D10, D21 to D11, D22 to D12, D23 to D13, D24 to D14, D25 to D15, D26 to D16, D27 to D17, D28 to D18, D29 to D19, D30 to D20, D31 to D21, D32 to D22, D33 to D23, D34 to D24, D5 to D4, D7 to D5, D8 to D6, D16 to D7, D17 to D8, D19 to D9, R20 to R10, R21 to R11, R22 to R12, R23 to R13, R24 to R14, R25 to R15, R26 to R16, R27 to R17, R28 to R18, R29 to R19, R30 to R20, R31 to R21, R32 to R22, R33 to R23, R4 to R3, R6 to R4, R7 to R5, R15 to R6, R16 to R7, R18 to R8, R19 to R9

Commit message: PCB MODIFIED INSIDE ONLYPINS
Parts:
- removed D23, D24: D_Zener, Diode_SMD:D_SOD-882, symbol Device:D_Zener
- removed J3, J5: Conn_01x19_Socket, Connector_PinHeader_2.54mm:PinHeader_1x19_P2.54mm_Vertical, symbol Connector:Conn_01x19_Socket
- removed R22, R23: 100, RC0805FR-07330RL:RESC2012X60N, symbol RC0805FR-07330RL:RC0805FR-07330RL
- added J6, J7: TB010-508-P19BK, TB010-508-P19BK:CUI_TB010-508-P19BK, symbol TB010-508-P19BK:TB010-508-P19BK
Connections:
- net IO16 is gone; now on net IO_16: R8.2
- net IO_0 is gone; now on net I/O_0: J2.6 (Pin_6)
- net IO_10 is gone; now on net SD3: J4.17 (Pin_17)
- net IO_11 is gone; now on net CMD: J4.18 (Pin_18)
- net IO_12 is gone; now on net I/O_12: J4.13 (Pin_13)
- net IO_15 is gone; now on net I/O_15: J2.4 (Pin_4)
- net IO_2 is gone; now on net I/O_2: J2.5 (Pin_5)
- net IO_36 is gone; now on net SP: J4.3 (Pin_3)
- net IO_39 is gone; now on net SN: J4.4 (Pin_4)
- net IO_5 is gone; now on net I/O_5: J2.10 (Pin_10)
- net IO_6 is gone; now on net CLK: J2.1 (Pin_1)
- net IO_7 is gone; now on net SD0: J2.2 (Pin_2)
- net IO_8 is gone; now on net SD1: J2.3 (Pin_3)
- net IO_9 is gone; now on net SD2: J4.16 (Pin_16)
- net +3V3: now also J6.1
- net CLK: now also J7.1
- net CMD: now also J6.18
- net EN: now also J6.2
- net GND: now also J6.14, J7.13, J7.19
- net I/O_0: now also J7.6
- net I/O_12: now also J6.13
- net I/O_13: now also J6.15
- net I/O_14: now also J6.12
- net I/O_15: now also J7.4
- net I/O_16: now also J7.8
- net I/O_17: now also J7.9
- net I/O_18: now also J7.11
- net I/O_19: now also J7.12
- net I/O_2: now also J7.5
- net I/O_21: now also J7.14
- net I/O_22: now also J7.17
- net I/O_23: now also J7.18
- net I/O_25: now also J6.9
- net I/O_26: now also J6.10
- net I/O_27: now also J6.11
- net I/O_32: now also J6.7
- net I/O_33: now also J6.8
- net I/O_34: now also J6.5
- net I/O_35: now also J6.6
- net I/O_4: now also J7.7
- net I/O_5: now also J7.10
- net RXD: now also J7.15
- net SD0: now also J7.2
- net SD1: now also J7.3
- net SD2: now also J6.16
- net SD3: now also J6.17
- net SN: now also J6.4
- net SP: now also J6.3
- net TXD: now also J7.16
- net VIN 5V: now also J6.19
Other:
- moved on the sheet: C1, C2, C3, C4, C5, C6, C7, C8, D1, D10, D11, D12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

Commit message: FINAL PCB WORK
Parts:
- removed D1: 1N5824, Diode_SMD:D_01005_0402Metric_Pad0.57x0.30mm_HandSolder, symbol Device:D
- added D1: 1N5824, 1N5824:DIOAD1898W129L762D1143, symbol 1N5824:1N5824
- renumbered J7 to J2, J2 to J3, J6 to J4, J4 to J5
Connections:
- net GND: now also D1.A
- net at L1.1, U1.2 (OUT): now also D1.C
