File: KiCad Projects/ESP32_PCB_ONLY_PINS/FINAL_DESIGN.kicad_sch (KiCad schematic)
At the start: 63 parts, among them J1 Screw_Terminal_01x02, J2 TB010-508-P19BK, J3 Conn_01x19_Socket, J4 TB010-508-P19BK, J5 Conn_01x19_Socket, Q1 PMOS, U1 LM2596S-5, U2 ESP32_NODEMCU

Commit message: PCB FINAL WORK DONE
Parts:
- removed D1: 1N5824, 1N5824:DIOAD1898W129L762D1143, symbol 1N5824:1N5824
- removed D10, D11, D12, D13, D14, D15, D16, D17, D18, D19, D20, D21, D22, D4, D5, D6, D7, D8, D9: D_Zener, Diode_SMD:D_SOD-882, symbol Device:D_Zener
- removed D2: D_Zener, Diode_THT:D_5W_P10.16mm_Horizontal, symbol Device:D_Zener
- removed Q1: PMOS, Package_TO_SOT_THT:TO-92L_HandSolder, symbol Simulation_SPICE:PMOS
- added CR1, CR10, CR11, CR12, CR13, CR14, CR15, CR16, CR17, CR18, CR19, CR2, CR3, CR4, CR5, CR6, CR7, CR8, CR9: PESD3V3L1BA_115, footprints:DIODE_PESD3V3L1BA_115_NEX, symbol 2026-03-30_09-39-47:PESD3V3L1BA_115
- added D1: SS34, SS34:DIO_SS34, symbol SS34:SS34
- added D2: MMBZ5242B-7-F, MMBZ5242B-7-F:SOT91P240X102-3N, symbol MMBZ5242B-7-F:MMBZ5242B-7-F
- added Q1: AO3401A, A03401:SOT23-3, symbol AO3401A:AO3401A
- C1: footprint Capacitor_THT:CP_Radial_D6.3mm_P2.50mm -> Capacitor_THT:CP_Radial_D10.0mm_P5.00mm
- C3: footprint Capacitor_THT:CP_Radial_D6.3mm_P2.50mm -> Capacitor_THT:CP_Radial_D8.0mm_P3.50mm
- C4, C7: footprint Capacitor_THT:C_Disc_D3.0mm_W2.0mm_P2.50mm -> Capacitor_SMD:C_0805_2012Metric
- C6, C8: footprint Capacitor_THT:C_Disc_D3.0mm_W1.6mm_P2.50mm -> Capacitor_SMD:C_0805_2012Metric
- J1: footprint TerminalBlock_4Ucon:TerminalBlock_4Ucon_1x02_P3.50mm_Vertical -> Connector_Phoenix_MC_HighVoltage:PhoenixContact_MCV_1,5_2-G-5.08_1x02_P5.08mm_Vertical
- R10, R11, R12, R13, R14, R15, R16, R17, R18, R19, R20, R21, R3, R4, R5, R6, R7, R8, R9: footprint RC0805FR-07330RL:RESC2012X60N -> Resistor_SMD:R_0805_2012Metric
- U2: now not fitted; now left out of the parts list
Connections:
- net 12V: now also D2.3, Q1.3
- net GND: now also CR1.2, CR10.2, CR11.2, CR12.2, CR13.2, CR14.2, CR15.2, CR16.2, CR17.2, CR18.2, CR19.2, CR2.2, CR3.2, CR4.2, CR5.2, CR6.2, CR7.2, CR8.2, CR9.2, D1.A, D2.1
- net I/O_13: now also CR4.1
- net I/O_14: now also CR5.1
- net I/O_16: now also CR6.1
- net I/O_17: now also CR7.1
- net I/O_18: now also CR8.1
- net I/O_19: now also CR9.1
- net I/O_21: now also CR10.1
- net I/O_22: now also CR11.1
- net I/O_23: now also CR12.1
- net I/O_25: now also CR13.1
- net I/O_26: now also CR14.1
- net I/O_27: now also CR15.1
- net I/O_32: now also CR16.1
- net I/O_33: now also CR17.1
- net I/O_34: now also CR18.1
- net I/O_35: now also CR19.1
- net I/O_4: now also CR3.1
- net RXD: now also CR2.1
- net TXD: now also CR1.1
- net at L1.1, U1.2 (OUT): now also D1.C
- net at F1.2, R1.1: now also Q1.2
- net at R1.2, R2.1: now also Q1.1
Other:
- moved on the sheet: R2
